Commit message: Fixed Bug in URDF

File: copernicus_description/urdf/accessories/wheel.urdf.xacro (robot description, xacro)
@@ -8,5 +8,5 @@
                 <origin xyz="0 0 0" rpy="${PI/2} 0 0"/>
                 <geometry>
-                    <mesh filename="$(find copernicus_description)/meshes/copernicus_wheel.STL"/>
+                    <mesh filename="package://copernicus_description/meshes/wheel.stl"/>
                 </geometry>
                 <material name="black"/>
@@ -19,9 +19,10 @@
             </collision>
             <inertial>
-                <origin xyz="0 0 0" rpy="${PI/2} 0 0"/>
-                <cylinder_inertia m="0.5" r="${wheel_radius}" h="${wheel_length}"/>
+                <mass value="2.637" />
+                <origin xyz="0 0 0" />
+                <inertia  ixx="0.02467" ixy="0" ixz="0" iyy="0.04411" iyz="0" izz="0.02467" />
             </inertial>
         </link>
-        <gazebo reference="$(wheel_prefix)_wheel">
+        <gazebo reference="${wheel_prefix}_wheel">
             <material>Gazebo/Black</material>
             <mu1 value="1.0"/>
@@ -32,5 +33,5 @@
         </gazebo>
         <!-- Wheel Joint -->
-        <joint name="$(wheel_prefix)_wheel_joint" type="continuous">
+        <joint name="${wheel_prefix}_wheel_joint" type="continuous">
             <parent link="base_link"/>
             <child link="${wheel_prefix}_wheel" />

File: copernicus_description/urdf/copernicus.urdf.xacro (robot description, xacro)
@@ -27,5 +27,5 @@
                 <origin xyz="0 0 0" rpy="0 0 0" />
                 <geometry>
-                    <mesh filename=""/>
+                    <mesh filename="package://copernicus_description/meshes/chassis.stl"/>
                 </geometry>
             </visual>
@@ -48,5 +48,5 @@
             <origin xyz="0 0 ${ wheel_joint_z - wheel_radius }" rpy="0 0 0" />
             <parent link="base_link" />
-            <child link="base_footprint" />
+            <child link="footprint" />
         </joint>
         <!-- Wheel -->

Commit message: Added new meshes and included in URDF

File: copernicus_description/urdf/accessories/wheel.urdf.xacro (robot description, xacro)
@@ -6,14 +6,14 @@
         <link name="${wheel_prefix}_wheel">
             <visual>
-                <origin xyz="0 0 0" rpy="${PI/2} 0 0"/>
+                <origin xyz="0 0 0" rpy="0 ${PI/2} 0"/>
                 <geometry>
-                    <mesh filename="package://copernicus_description/meshes/wheel.stl"/>
+                    <mesh filename="package://copernicus_description/meshes/wheel.STL"/>
                 </geometry>
                 <material name="black"/>
             </visual>
             <collision>
-                <origin xyz="0 0 0" rpy="${PI/2} 0 0"/>
+                <origin xyz="0 0 0" rpy="0 ${PI/2} 0"/>
                 <geometry>
-                    <cylinder length="${wheel_length}" radius="${wheel_radius}"/>
+                    <cylinder length="${wheel_width}" radius="${wheel_radius}"/>
                 </geometry>
             </collision>

File: copernicus_description/urdf/copernicus.urdf.xacro (robot description, xacro)
@@ -6,13 +6,17 @@
     <!-- xacro properties -->
     <xacro:property name="PI" value="3.14159"/>
-    <xacro:property name="base_mass" value="27.2155"/>
-    <xacro:property name="base_l" value="0.74"/>
-    <xacro:property name="base_w" value="0.42"/>
-    <xacro:property name="base_h" value="0.32"/>
-    <xacro:property name="wheel_length" value="0.1143" />
+    <xacro:property name="chassis_mass" value="48.00"/>
+    <xacro:property name="chassis_l" value="0.75"/>
+    <xacro:property name="chassis_w" value="0.42"/>
+    <xacro:property name="chassis_h" value="0.23042"/>
+    <xacro:property name="chassis_h_no_susp" value="0.14"/>
+    <xacro:property name="chassis_t" value="0.003"/>
+    <xacro:property name="body_mass" value="11.869"/>
+    <xacro:property name="body_h" value="0.15"/>
+    <xacro:property name="wheel_width" value="0.1143" />
     <xacro:property name="wheel_radius" value="0.16" />
-    <xacro:property name="wheel_joint_x" value="0.26" />
-    <xacro:property name="wheel_joint_y" value="0.21" />
-    <xacro:property name="wheel_joint_z" value="0.16" />
+    <xacro:property name="wheel_joint_x" value="0.02" />
+    <xacro:property name="wheel_joint_y" value="0.11233" />
+    <xacro:property name="wheel_joint_z" value="-0.04295" />
     <xacro:property name="dummy_inertia" value="1e-09"/>
     <!-- xacro args -->
@@ -22,44 +26,69 @@
     <xacro:arg name="camera_enabled" default="false"/>
     <xacro:macro name="copernicus_robot">
-        <!-- Base link -->
+        <!-- Chassis aka base link -->
         <link name="base_link">
             <visual>
                 <origin xyz="0 0 0" rpy="0 0 0" />
                 <geometry>
-                    <mesh filename="package://copernicus_description/meshes/chassis.stl"/>
+                    <mesh filename="package://copernicus_description/meshes/chassis.STL"/>
                 </geometry>
             </visual>
             <collision>
-                <origin xyz="0 0 ${base_h/4}" rpy="0 0 0" />
+                <origin xyz="0 0 0" rpy="0 0 0" />
                 <geometry>
-                    <box size="${base_l} ${base_w} ${base_h/2}"/>
+                    <box size="${chassis_l} ${chassis_w} ${chassis_h}"/>
                 </geometry>
             </collision>
-            <collision>
-                <origin xyz="0 0 ${base_h*3/4}" rpy="0 0 0" />
-                <geometry>
-                    <box size="${base_l*4/5} ${base_w} ${base_h/2}"/>
-                </geometry>
-            </collision>
+	    <inertial>
+	    	<mass value="${chassis_mass}"/>
+		<inertia ixx="2.762187" ixy="-1.06570" ixz="-0.87376" iyy="0.99303" iyz="0.15602" izz="3.65234"/>
+	    </inertial>
         </link>
+	<!-- Body assembly -->
+	<link name="body">
+		<visual>
+			<geometry>
+				<mesh filename="package://copernicus_description/meshes/body.STL"/>
+			</geometry>
+			<origin xyz="0 0 0" rpy="0 ${PI/2} 0"/>
+		</visual>
+		<collision>
+			<geometry>
+				<box size="${chassis_l} ${chassis_w} ${body_h}"/>
+			</geometry>
+			<origin xyz="0 0 0" rpy="0 ${PI/2} 0"/>
+		</collision>
+		<inertial>
+			<mass value="${body_mass}"/>
+			<inertia ixx="3.076852" ixy="-0.33079" ixz="0.1645412" iyy="0.82521" iyz="-0.95871" izz="2.42356"/>
+		</inertial>
+	</link>
         <!-- Footprint -->
         <link name="footprint"/>
+	<!-- Joints -->
+	<!-- Joint from footprint to base link(chassis) -->
         <joint name="base_footprint_joint" type="fixed">
-            <origin xyz="0 0 ${ wheel_joint_z - wheel_radius }" rpy="0 0 0" />
+            <origin xyz="0 0 ${-wheel_radius+wheel_joint_z}" rpy="0 0 0" />
             <parent link="base_link" />
             <child link="footprint" />
         </joint>
+	<!-- Joint between chassis and body -->
+	<joint name="chassis_body_joint" type="fixed">
+		<parent link="base_link"/>
+		<child link="body"/>
+		<origin xyz="${-2*chassis_t} 0 ${chassis_h_no_susp}" rpy="0 0 0"/>
+	</joint>
         <!-- Wheel -->
         <xacro:copernicus_wheel wheel_prefix="front_left">
-            <origin xyz="${wheel_joint_x} ${wheel_joint_y} ${wheel_joint_z}" rpy="0 0 0" />
+            <origin xyz="${wheel_joint_x+wheel_width} ${wheel_joint_y} ${wheel_joint_z}" rpy="0 0 0" />
         </xacro:copernicus_wheel>
         <xacro:copernicus_wheel wheel_prefix="front_right">
-            <origin xyz="${wheel_joint_x} ${-wheel_joint_y} ${wheel_joint_z}" rpy="0 0 0" />
+            <origin xyz="${-(wheel_joint_x+chassis_w)} ${wheel_joint_y} ${wheel_joint_z}" rpy="0 0 0" />
         </xacro:copernicus_wheel>
         <xacro:copernicus_wheel wheel_prefix="back_left">
-            <origin xyz="${-wheel_joint_x} ${wheel_joint_y} ${wheel_joint_z}" rpy="0 0 0" />
+            <origin xyz="${wheel_joint_x+wheel_width} ${chassis_l-wheel_joint_y} ${wheel_joint_z}" rpy="0 0 0" />
         </xacro:copernicus_wheel>
         <xacro:copernicus_wheel wheel_prefix="back_right">
-            <origin xyz="${-wheel_joint_x} ${-wheel_joint_y} ${wheel_joint_z}" rpy="0 0 0" />
+            <origin xyz="${-(wheel_joint_x+chassis_w)} ${chassis_l-wheel_joint_y} ${wheel_joint_z}" rpy="0 0 0" />
         </xacro:copernicus_wheel>
         <!-- LIDAR -->

Commit message: Changed coordinate systems of STLs

File: copernicus_description/urdf/accessories/wheel.urdf.xacro (robot description, xacro)
@@ -6,5 +6,5 @@
         <link name="${wheel_prefix}_wheel">
             <visual>
-                <origin xyz="0 0 0" rpy="0 ${PI/2} 0"/>
+                <origin xyz="0 0 0" rpy="0 0 0"/>
                 <geometry>
                     <mesh filename="package://copernicus_description/meshes/wheel.STL"/>
@@ -13,7 +13,7 @@
             </visual>
             <collision>
-                <origin xyz="0 0 0" rpy="0 ${PI/2} 0"/>
+                <origin xyz="0 0 0" rpy="0 0 0"/>
                 <geometry>
-                    <cylinder length="${wheel_width}" radius="${wheel_radius}"/>
+			<mesh filename="package://copernicus_description/meshes/wheel.STL"/>
                 </geometry>
             </collision>

File: copernicus_description/urdf/copernicus.urdf.xacro (robot description, xacro)
@@ -16,7 +16,7 @@
     <xacro:property name="wheel_width" value="0.1143" />
     <xacro:property name="wheel_radius" value="0.16" />
-    <xacro:property name="wheel_joint_x" value="0.02" />
-    <xacro:property name="wheel_joint_y" value="0.11233" />
-    <xacro:property name="wheel_joint_z" value="-0.04295" />
+    <xacro:property name="wheel_joint_x_abs" value="0.28908" />
+    <xacro:property name="wheel_joint_y_abs" value="0.26267" />
+    <xacro:property name="wheel_joint_z_abs" value="0.04795" />
     <xacro:property name="dummy_inertia" value="1e-09"/>
     <!-- xacro args -->
@@ -25,4 +25,13 @@
     <xacro:arg name="gps_enabled" default="false"/>
     <xacro:arg name="camera_enabled" default="false"/>
+    <material name="blue">
+	<color rgba="0 0 0.8 1"/>
+    </material>
+    <material name="white">
+	<color rgba="1 1 1 1"/>
+    </material>
+    <material name="gray">
+	<color rgba="0.5 0.5 0.5 1"/>
+    </material>
     <xacro:macro name="copernicus_robot">
         <!-- Chassis aka base link -->
@@ -33,9 +42,10 @@
                     <mesh filename="package://copernicus_description/meshes/chassis.STL"/>
                 </geometry>
+		<material name="gray"/>
             </visual>
             <collision>
                 <origin xyz="0 0 0" rpy="0 0 0" />
                 <geometry>
-                    <box size="${chassis_l} ${chassis_w} ${chassis_h}"/>
+			<mesh filename="package://copernicus_description/meshes/chassis.STL"/>
                 </geometry>
             </collision>
@@ -51,11 +61,12 @@
 				<mesh filename="package://copernicus_description/meshes/body.STL"/>
 			</geometry>
-			<origin xyz="0 0 0" rpy="0 ${PI/2} 0"/>
+			<origin xyz="0 0 0" rpy="0 0 0"/>
+			<material name="white"/>
 		</visual>
 		<collision>
 			<geometry>
-				<box size="${chassis_l} ${chassis_w} ${body_h}"/>
+				<mesh filename="package://copernicus_description/meshes/body.STL"/>
 			</geometry>
-			<origin xyz="0 0 0" rpy="0 ${PI/2} 0"/>
+			<origin xyz="0 0 0" rpy="0 0 0"/>
 		</collision>
 		<inertial>
@@ -69,5 +80,5 @@
 	<!-- Joint from footprint to base link(chassis) -->
         <joint name="base_footprint_joint" type="fixed">
-            <origin xyz="0 0 ${-wheel_radius+wheel_joint_z}" rpy="0 0 0" />
+            <origin xyz="0 0 ${-((wheel_joint_z_abs-chassis_h_no_susp)+2*wheel_radius)}" rpy="0 0 0" />
             <parent link="base_link" />
             <child link="footprint" />
@@ -77,18 +88,18 @@
 		<parent link="base_link"/>
 		<child link="body"/>
-		<origin xyz="${-2*chassis_t} 0 ${chassis_h_no_susp}" rpy="0 0 0"/>
+		<origin xyz="0 0 ${chassis_h_no_susp-0.005}" rpy="0 0 0"/>
 	</joint>
         <!-- Wheel -->
         <xacro:copernicus_wheel wheel_prefix="front_left">
-            <origin xyz="${wheel_joint_x+wheel_width} ${wheel_joint_y} ${wheel_joint_z}" rpy="0 0 0" />
+            <origin xyz="${wheel_joint_x_abs} ${-wheel_joint_y_abs} ${-wheel_joint_z_abs}" rpy="0 0 0" />
         </xacro:copernicus_wheel>
         <xacro:copernicus_wheel wheel_prefix="front_right">
-            <origin xyz="${-(wheel_joint_x+chassis_w)} ${wheel_joint_y} ${wheel_joint_z}" rpy="0 0 0" />
+            <origin xyz="${-wheel_joint_x_abs} ${-wheel_joint_y_abs} ${-wheel_joint_z_abs}" rpy="0 0 0" />
         </xacro:copernicus_wheel>
         <xacro:copernicus_wheel wheel_prefix="back_left">
-            <origin xyz="${wheel_joint_x+wheel_width} ${chassis_l-wheel_joint_y} ${wheel_joint_z}" rpy="0 0 0" />
+            <origin xyz="${wheel_joint_x_abs} ${wheel_joint_y_abs} ${-wheel_joint_z_abs}" rpy="0 0 0" />
         </xacro:copernicus_wheel>
         <xacro:copernicus_wheel wheel_prefix="back_right">
-            <origin xyz="${-(wheel_joint_x+chassis_w)} ${chassis_l-wheel_joint_y} ${wheel_joint_z}" rpy="0 0 0" />
+            <origin xyz="${-wheel_joint_x_abs} ${wheel_joint_y_abs} ${-wheel_joint_z_abs}" rpy="0 0 0" />
         </xacro:copernicus_wheel>
         <!-- LIDAR -->

Commit message: Fixed Orientation of STL Files

File: copernicus_description/urdf/accessories/wheel.urdf.xacro (robot description, xacro)
@@ -6,5 +6,5 @@
         <link name="${wheel_prefix}_wheel">
             <visual>
-                <origin xyz="0 0 0" rpy="0 0 0"/>
+                <origin xyz="0 0 0" rpy="0 0 ${PI/2}"/>
                 <geometry>
                     <mesh filename="package://copernicus_description/meshes/wheel.STL"/>
@@ -13,5 +13,5 @@
             </visual>
             <collision>
-                <origin xyz="0 0 0" rpy="0 0 0"/>
+                <origin xyz="0 0 0" rpy="0 0 ${PI/2}"/>
                 <geometry>
 			<mesh filename="package://copernicus_description/meshes/wheel.STL"/>

Commit message: Updated Description to Match ros_control specs

File: copernicus_description/urdf/accessories/wheel.urdf.xacro (robot description, xacro)
@@ -13,7 +13,7 @@
             </visual>
             <collision>
-                <origin xyz="0 0 0" rpy="0 0 ${PI/2}"/>
+                <origin xyz="0 0 0" rpy="${PI/2} 0 0"/>
                 <geometry>
-			<mesh filename="package://copernicus_description/meshes/wheel.STL"/>
+                    <cylinder length="${wheel_width}" radius="${wheel_radius+0.01}" />
                 </geometry>
             </collision>
@@ -28,7 +28,4 @@
             <mu1 value="1.0"/>
             <mu2 value="1.0"/>
-            <kp value="10000000.0" />
-            <kd value="1.0" />
-            <fdir1 value="1 0 0"/>
         </gazebo>
         <!-- Wheel Joint -->
@@ -43,5 +40,5 @@
             <type>transmission_interface/SimpleTransmission</type>
             <joint name="${wheel_prefix}_wheel_joint">
-                <hardwareInterface>VelocityJointInterface</hardwareInterface>
+                <hardwareInterface>hardware_interface/VelocityJointInterface</hardwareInterface>
             </joint>
             <actuator name="${wheel_prefix}_motor">

File: copernicus_description/urdf/copernicus.urdf.xacro (robot description, xacro)
@@ -55,28 +55,28 @@
 	    </inertial>
         </link>
-	<!-- Body assembly -->
-	<link name="body">
-		<visual>
-			<geometry>
-				<mesh filename="package://copernicus_description/meshes/body.STL"/>
-			</geometry>
-			<origin xyz="0 0 0" rpy="0 0 0"/>
-			<material name="white"/>
-		</visual>
-		<collision>
-			<geometry>
-				<mesh filename="package://copernicus_description/meshes/body.STL"/>
-			</geometry>
-			<origin xyz="0 0 0" rpy="0 0 0"/>
-		</collision>
-		<inertial>
-			<mass value="${body_mass}"/>
-			<inertia ixx="3.076852" ixy="-0.33079" ixz="0.1645412" iyy="0.82521" iyz="-0.95871" izz="2.42356"/>
-		</inertial>
-	</link>
+        <!-- Body assembly -->
+        <link name="body">
+            <visual>
+                <geometry>
+                    <mesh filename="package://copernicus_description/meshes/body.STL"/>
+                </geometry>
+                <origin xyz="0 0 0" rpy="0 0 0"/>
+                <material name="white"/>
+            </visual>
+            <collision>
+                <geometry>
+                    <mesh filename="package://copernicus_description/meshes/body.STL"/>
+                </geometry>
+                <origin xyz="0 0 0" rpy="0 0 0"/>
+            </collision>
+            <inertial>
+                <mass value="${body_mass}"/>
+                <inertia ixx="3.076852" ixy="-0.33079" ixz="0.1645412" iyy="0.82521" iyz="-0.95871" izz="2.42356"/>
+            </inertial>
+        </link>
         <!-- Footprint -->
         <link name="footprint"/>
-	<!-- Joints -->
-	<!-- Joint from footprint to base link(chassis) -->
+        <!-- Joints -->
+        <!-- Joint from footprint to base link(chassis) -->
         <joint name="base_footprint_joint" type="fixed">
             <origin xyz="0 0 ${-((wheel_joint_z_abs-chassis_h_no_susp)+2*wheel_radius)}" rpy="0 0 0" />
@@ -84,21 +84,21 @@
             <child link="footprint" />
         </joint>
-	<!-- Joint between chassis and body -->
-	<joint name="chassis_body_joint" type="fixed">
-		<parent link="base_link"/>
-		<child link="body"/>
-		<origin xyz="0 0 ${chassis_h_no_susp-0.005}" rpy="0 0 0"/>
-	</joint>
+        <!-- Joint between chassis and body -->
+        <joint name="chassis_body_joint" type="fixed">
+            <parent link="base_link"/>
+            <child link="body"/>
+            <origin xyz="0 0 ${chassis_h_no_susp-0.005}" rpy="0 0 0"/>
+        </joint>
         <!-- Wheel -->
+        <xacro:copernicus_wheel wheel_prefix="front_right">
+            <origin xyz="${wheel_joint_x_abs} ${-wheel_joint_y_abs} ${-wheel_joint_z_abs}" rpy="0 0 0" />
+        </xacro:copernicus_wheel>
+        <xacro:copernicus_wheel wheel_prefix="back_right">
+            <origin xyz="${-wheel_joint_x_abs} ${-wheel_joint_y_abs} ${-wheel_joint_z_abs}" rpy="0 0 0" />
+        </xacro:copernicus_wheel>
         <xacro:copernicus_wheel wheel_prefix="front_left">
-            <origin xyz="${wheel_joint_x_abs} ${-wheel_joint_y_abs} ${-wheel_joint_z_abs}" rpy="0 0 0" />
-        </xacro:copernicus_wheel>
-        <xacro:copernicus_wheel wheel_prefix="front_right">
-            <origin xyz="${-wheel_joint_x_abs} ${-wheel_joint_y_abs} ${-wheel_joint_z_abs}" rpy="0 0 0" />
+            <origin xyz="${wheel_joint_x_abs} ${wheel_joint_y_abs} ${-wheel_joint_z_abs}" rpy="0 0 0" />
         </xacro:copernicus_wheel>
         <xacro:copernicus_wheel wheel_prefix="back_left">
-            <origin xyz="${wheel_joint_x_abs} ${wheel_joint_y_abs} ${-wheel_joint_z_abs}" rpy="0 0 0" />
-        </xacro:copernicus_wheel>
-        <xacro:copernicus_wheel wheel_prefix="back_right">
             <origin xyz="${-wheel_joint_x_abs} ${wheel_joint_y_abs} ${-wheel_joint_z_abs}" rpy="0 0 0" />
         </xacro:copernicus_wheel>
@@ -106,12 +106,4 @@
             <plugin name="gazebo_ros_control" filename="libgazebo_ros_control.so">
                 <robotNamespace>/</robotNamespace>
-            </plugin>
-            <plugin name="omni_steering" filename="libgazebo_ros_planar_move.so">
-                <robotNamespace>/</robotNamespace>
-                <commandTopic>cmd_vel</commandTopic>
-                <odometryTopic>odometry/wheel</odometryTopic>
-                <odometryFrame>odom</odometryFrame>
-                <odometryRate>30.0</odometryRate>
-                <robotBaseFrame>footprint</robotBaseFrame>
             </plugin>
         </gazebo>
