Commit message: Modified Accessories XACROs

File: copernicus_description/urdf/accessories/camera.urdf.xacro (robot description, xacro)
@@ -1,2 +1,3 @@
+<?xml version="1.0"?>
 <!--
 Copyright (c) 2017, Botsync Pte. Ltd.
@@ -23,14 +24,13 @@
 SOFTWARE, EVEN IF ADVISED OF THE POSSIBILITY OF SUCH DAMAGE.
 -->
-<?xml version="1.0"?>
+<!-- TODO: Camera Mesh, Mount and Origin -->
 <robot name="copernicus" xmlns:xacro="https://ros.org/wiki/xacro">
-    <xacro:macro name="camera" params="frame:=camera topic:=camera info_topic:=camera_info update_rate:=50 robot_namespace:=/">
+    <xacro:macro name="camera_" params="frame:=camera topic:=camera info_topic:=camera_info update_rate:=50 robot_namespace:=/">
+        <joint name="base_to_camera" type="fixed">
+            <parent link="base_link"/>
+            <child link="${frame}"/>
+            <origin xyz="0 0 ${chassis_h}"/>
+        </joint>
         <link name="${frame}">
-            <collision>
-                <origin xyz="0 0 0" rpy="0 0 0"/>
-                <geometry>
-                    <mesh filename="package://copernicus_description/meshes/logitech_c910.stl"/>
-                </geometry>
-            </collision>
             <visual>
                 <origin xyz="0 0 0" rpy="0 0 0"/>
@@ -38,6 +38,11 @@
                     <box size="0.07 0.09 0.07"/>
                 </geometry>
-                <material name="black"/>
             </visual>
+            <collision>
+                <origin xyz="0 0 0" rpy="0 0 0"/>
+                <geometry>
+                    <box size="0.07 0.09 0.07"/>
+                </geometry>
+            </collision>
             <inertial>
                 <mass value="0.162"/>
@@ -46,11 +51,5 @@
             </inertial>
         </link>
-        <joint name="base_to_camera" type="fixed">
-            <parent link="base_link"/>
-            <child link="${frame}"/>
-            <origin xyz="${ 0.0 } ${ 0.0 } ${ 0.0 }"/>
-        </joint>
         <gazebo reference="${frame}">
-            <material>Gazebo/Blue</material>
             <sensor type="camera" name="camera">
                 <update_rate>${update_rate}</update_rate>
@@ -66,4 +65,9 @@
                     <far>300</far>
                     </clip>
+                    <noise>
+                      <type>gaussian</type>
+                      <mean>0.0</mean>
+                      <stddev>0.007</stddev>
+                    </noise>
                 </camera>
                 <plugin name="camera_controller" filename="libgazebo_ros_camera.so">

File: copernicus_description/urdf/accessories/gps.urdf.xacro (robot description, xacro)
@@ -1,2 +1,3 @@
+<?xml version="1.0"?>
 <!--
 Copyright (c) 2017, Botsync Pte. Ltd.
@@ -23,5 +24,4 @@
 SOFTWARE, EVEN IF ADVISED OF THE POSSIBILITY OF SUCH DAMAGE.
 -->
-<?xml version="1.0"?>
 <robot name="copernicus" xmlns:xacro="https://ros.org/wiki/xacro">
     <xacro:macro name="gps" params="frame:=gps topic:=gps/fix update_rate:=50 robot_namespace:=/ refLat:=1.345490 refLong:=103.682360">
@@ -37,7 +37,7 @@
             <child link="${frame}" />
         </joint>
-        <gazebo reference="${frame}">
+        <gazebo>
             <plugin name="gps_plugin" filename="libhector_gazebo_ros_gps.so">
-                <robotNamespace>${ robot_namespace }</robotNamespace>
+                <robotNamespace>${robot_namespace}</robotNamespace>
                 <updateRate>${update_rate}</updateRate>
                 <bodyName>${frame}</bodyName>

File: copernicus_description/urdf/accessories/imu.urdf.xacro (robot description, xacro)
@@ -1,2 +1,3 @@
+<?xml version="1.0"?>
 <!--
 Copyright (c) 2017, Botsync Pte. Ltd.
@@ -23,19 +24,19 @@
 SOFTWARE, EVEN IF ADVISED OF THE POSSIBILITY OF SUCH DAMAGE.
 -->
-<?xml version="1.0"?>
 <robot name="copernicus" xmlns:xacro="https://ros.org/wiki/xacro">
     <xacro:macro name="imu" params="frame:=imu topic:=imu/data update_rate:=50 robot_namespace:=/">
+        <joint name="${frame}_joint" type="fixed">
+            <parent link="base_link" />
+            <child link="${frame}" />
+            <origin xyz="0 0 ${chassis_h_no_susp/2}" rpy="0 0 0" />
+        </joint>
         <link name="${frame}">
             <inertial>
                 <mass value="0.001"/>
                 <origin xyz="0 0 0" rpy="0 0 0"/>
-                <inertia ixx="${dummy_inertia}" ixy="0.0" ixz="0.0" iyy="${dummy_inertia}" iyz="0.0" izz="${dummy_inertia}"/>
+                <inertia ixx="1e-09" ixy="0.0" ixz="0.0" iyy="1e-09" iyz="0.0" izz="1e-09"/>
             </inertial>
         </link>
-        <joint name="${frame}_joint" type="fixed">
-            <parent link="base_link" />
-            <child link="${frame}" />
-        </joint>
-        <gazebo reference="${frame}">
+        <gazebo>
             <plugin name="imu_plugin" filename="libhector_gazebo_ros_imu.so">
                 <robotNamespace>${robot_namespace}</robotNamespace>
@@ -47,5 +48,5 @@
                 <accelGaussianNoise>0.005 0.005 0.005</accelGaussianNoise>
                 <rateDrift>0.005 0.005 0.005 </rateDrift>
-                <rateGaussianNoise>0.005 0.005 0.005 </rateGaussianNoise>
+                <rateGaussianNoise>0.005 0.005 0.005</rateGaussianNoise>
                 <headingDrift>0.005</headingDrift>
                 <headingGaussianNoise>0.005</headingGaussianNoise>

File: copernicus_description/urdf/accessories/lidar.urdf.xacro (robot description, xacro)
@@ -1,2 +1,3 @@
+<?xml version="1.0"?>
 <!--
 Copyright (c) 2017, Botsync Pte. Ltd.
@@ -23,5 +24,4 @@
 SOFTWARE, EVEN IF ADVISED OF THE POSSIBILITY OF SUCH DAMAGE.
 -->
-<?xml version="1.0"?>
 <robot name="copernicus" xmlns:xacro="https://ros.org/wiki/xacro">
   <xacro:macro name="lidar" params="frame:=lidar topic:=scan sample_size:=720 update_rate:=50
@@ -80,5 +80,4 @@
       </link>
       <gazebo reference="${frame}">
-        <turnGravityOff>true</turnGravityOff>
         <sensor type="ray" name="${frame}">
           <pose>0 0 0 0 0 0</pose>

File: copernicus_description/urdf/components/wheel.urdf.xacro (robot description, xacro)
@@ -1,2 +1,3 @@
+<?xml version="1.0"?>
 <!--
 Copyright (c) 2017, Botsync Pte. Ltd.
@@ -23,5 +24,4 @@
 SOFTWARE, EVEN IF ADVISED OF THE POSSIBILITY OF SUCH DAMAGE.
 -->
-<?xml version="1.0"?>
 <robot name="copernicus_wheel" xmlns:xacro="https://ros.org/wiki/xacro">
     <!-- Wheel Macro -->

File: copernicus_description/urdf/copernicus.urdf.xacro (robot description, xacro)
@@ -1,2 +1,3 @@
+<?xml version="1.0"?>
 <!--
 Copyright (c) 2017, Botsync Pte. Ltd.
@@ -23,5 +24,4 @@
 SOFTWARE, EVEN IF ADVISED OF THE POSSIBILITY OF SUCH DAMAGE.
 -->
-<?xml version="1.0"?>
 <robot name="copernicus_robot" xmlns:xacro="https://ros.org/wiki/xacro">
     <!-- xacro includes -->
@@ -32,16 +32,8 @@
     <!-- xacro args -->
     <xacro:arg name="lidar_enabled" default="true"/>
-    <xacro:arg name="imu_enabled" default="false"/>
+    <xacro:arg name="imu_enabled" default="true"/>
     <xacro:arg name="gps_enabled" default="false"/>
+    <!-- TODO: Camera Mesh, Mount and Origin -->
     <xacro:arg name="camera_enabled" default="false"/>
-    <material name="blue">
-        <color rgba="0 0 0.8 1"/>
-    </material>
-    <material name="white">
-       <color rgba="1 1 1 1"/>
-    </material>
-    <material name="gray">
-        <color rgba="0.5 0.5 0.5 1"/>
-    </material>
     <xacro:macro name="copernicus_robot">
         <!-- Footprint -->
@@ -127,13 +119,13 @@
             </plugin>
         </gazebo>
+        <!-- IMU -->
+        <xacro:if value="$(arg imu_enabled)">
+            <xacro:include filename="$(find copernicus_description)/urdf/accessories/imu.urdf.xacro"/>
+            <xacro:imu></xacro:imu>
+        </xacro:if>
         <!-- LIDAR -->
         <xacro:if value="$(arg lidar_enabled)">
             <xacro:include filename="$(find copernicus_description)/urdf/accessories/lidar.urdf.xacro"/>
             <xacro:lidar></xacro:lidar>
-        </xacro:if>
-        <!-- IMU -->
-        <xacro:if value="$(arg imu_enabled)">
-            <xacro:include filename="$(find copernicus_description)/urdf/accessories/imu.urdf.xacro"/>
-            <xacro:imu></xacro:imu>
         </xacro:if>
         <!-- GPS -->
@@ -143,7 +135,8 @@
         </xacro:if>
         <!-- Camera -->
+        <!-- TODO: Camera Mesh, Mount and Origin -->
         <xacro:if value="$(arg camera_enabled)">
             <xacro:include filename="$(find copernicus_description)/urdf/accessories/camera.urdf.xacro"/>
-            <xacro:camera></xacro:camera>
+            <xacro:camera_></xacro:camera_>
         </xacro:if>
     </xacro:macro>

File: copernicus_description/urdf/vehicle_properties.xacro (robot description, xacro)
@@ -1,2 +1,3 @@
+<?xml version="1.0"?>
 <!--
 Copyright (c) 2017, Botsync Pte. Ltd.
@@ -23,6 +24,14 @@
 SOFTWARE, EVEN IF ADVISED OF THE POSSIBILITY OF SUCH DAMAGE.
 -->
-<?xml version="1.0"?>
 <robot name="copernicus_robot" xmlns:xacro="https://ros.org/wiki/xacro">
+    <material name="blue">
+        <color rgba="0 0 0.8 1"/>
+    </material>
+    <material name="white">
+       <color rgba="1 1 1 1"/>
+    </material>
+    <material name="gray">
+        <color rgba="0.5 0.5 0.5 1"/>
+    </material>
     <xacro:property name="chassis_mass" value="5.674"/>
     <xacro:property name="chassis_l" value="0.75"/>

Commit message: Updated urdf file of copernicus_v1

File: copernicus_description/urdf/accessories/camera.urdf.xacro (robot description, xacro)
@@ -30,5 +30,5 @@
             <parent link="base_link"/>
             <child link="${frame}"/>
-            <origin xyz="0 0 ${chassis_h}"/>
+            <origin xyz="0 0 ${base_h}"/>
         </joint>
         <link name="${frame}">

File: copernicus_description/urdf/accessories/imu.urdf.xacro (robot description, xacro)
@@ -29,5 +29,5 @@
             <parent link="base_link" />
             <child link="${frame}" />
-            <origin xyz="0 0 ${chassis_h_no_susp/2}" rpy="0 0 0" />
+            <origin xyz="0 0 ${base_h/2}" rpy="0 0 0" />
         </joint>
         <link name="${frame}">

File: copernicus_description/urdf/accessories/lidar.urdf.xacro (robot description, xacro)
@@ -28,5 +28,5 @@
                  min_angle:=-2.35619 max_angle:=2.35619 min_range:=0.5 max_range:=20.0 robot_namespace:=/">
       <joint name="lidar_mount_joint" type="fixed">
-          <origin xyz="${chassis_l/2} 0 0.035" rpy="0 0 0" />
+          <origin xyz="${lidar_mount_joint_x} ${lidar_mount_joint_y} ${lidar_mount_joint_z}" rpy="0 0 0" />
           <parent link="base_link" />
           <child link="lidar_mount" />
@@ -49,9 +49,9 @@
               <origin xyz="0 0 0" rpy="0 0 0"/>
               <mass value="0.1"/>
-              <inertia ixx="${dummy_inertia}" ixy="0.0" ixz="0.0" iyy="${dummy_inertia}" iyz="0.0" izz="${dummy_inertia}" />
+              <inertia ixx="${lidar_mount_ixx}" ixy="${lidar_mount_ixy}" ixz="${lidar_mount_ixz}" iyy="${lidar_mount_iyy}" iyz="${lidar_mount_iyz}" izz="${lidar_mount_izz}" />
           </inertial>
       </link>
       <joint name="lidar_joint" type="fixed">
-          <origin xyz="0.01 0 0" rpy="${PI} 0 0" />
+          <origin xyz="${lidar_joint_x} 0 0" rpy="${PI} 0 0" />
           <parent link="lidar_mount" />
           <child link="${frame}" />

File: copernicus_description/urdf/copernicus.urdf.xacro (robot description, xacro)
@@ -41,5 +41,5 @@
         <!-- Joint from footprint to base link(chassis) -->
         <joint name="base_footprint_joint" type="fixed">
-            <origin xyz="0 0 ${-(wheel_joint_z_abs+wheel_radius)}" rpy="0 0 0" />
+            <origin xyz="0 0 ${-base_underside_h}" rpy="0 0 0" />
             <parent link="base_link" />
             <child link="footprint" />
@@ -50,5 +50,5 @@
                 <origin xyz="0 0 0" rpy="0 0 0" />
                 <geometry>
-                    <mesh filename="package://copernicus_description/meshes/chassis.STL"/>
+                    <mesh filename="package://copernicus_description/meshes/copernicus.STL"/>
                 </geometry>
                 <material name="gray"/>
@@ -57,50 +57,24 @@
                 <origin xyz="0 0 0" rpy="0 0 0" />
                 <geometry>
-                    <mesh filename="package://copernicus_description/meshes/chassis.STL"/>
+                    <mesh filename="package://copernicus_description/meshes/copernicus.STL"/>
                 </geometry>
             </collision>
             <inertial>
-                <mass value="${ chassis_mass }"/>
-                <inertia ixx="${chassis_ixx}" ixy="${chassis_ixy}" ixz="${chassis_ixz}" iyy="${chassis_iyy}" iyz="${chassis_iyz}" izz="${chassis_izz}"/>
-            </inertial>
-        </link>
-        <!-- Joint between chassis and body -->
-        <joint name="chassis_body_joint" type="fixed">
-            <parent link="base_link"/>
-            <child link="body"/>
-            <origin xyz="0 0 ${chassis_h_no_susp-0.005}" rpy="0 0 0"/>
-        </joint>
-        <!-- Body assembly -->
-        <link name="body">
-            <visual>
-                <geometry>
-                    <mesh filename="package://copernicus_description/meshes/body.STL"/>
-                </geometry>
-                <origin xyz="0 0 0" rpy="0 0 0"/>
-                <material name="white"/>
-            </visual>
-            <collision>
-                <geometry>
-                    <mesh filename="package://copernicus_description/meshes/body.STL"/>
-                </geometry>
-                <origin xyz="0 0 0" rpy="0 0 0"/>
-            </collision>
-            <inertial>
-                <mass value="${body_mass}"/>
-                <inertia ixx="${body_ixx}" ixy="${body_ixy}" ixz="${body_ixz}" iyy="${body_iyy}" iyz="${body_iyz}" izz="${body_izz}"/>
+                <mass value="${base_mass }"/>
+                <inertia ixx="${base_ixx}" ixy="${base_ixy}" ixz="${base_ixz}" iyy="${base_iyy}" iyz="${base_iyz}" izz="${base_izz}"/>
             </inertial>
         </link>
         <!-- Wheel -->
         <xacro:copernicus_wheel wheel_prefix="front_right">
-            <origin xyz="${wheel_joint_x_abs} ${-wheel_joint_y_abs} ${-wheel_joint_z_abs}" rpy="0 0 0" />
+            <origin xyz="${wheel_front_joint_x_abs} ${-wheel_joint_y_abs} ${-wheel_joint_z_abs}" rpy="0 0 0" />
         </xacro:copernicus_wheel>
         <xacro:copernicus_wheel wheel_prefix="back_right">
-            <origin xyz="${-wheel_joint_x_abs} ${-wheel_joint_y_abs} ${-wheel_joint_z_abs}" rpy="0 0 0" />
+            <origin xyz="${-wheel_back_joint_x_abs} ${-wheel_joint_y_abs} ${-wheel_joint_z_abs}" rpy="0 0 0" />
         </xacro:copernicus_wheel>
         <xacro:copernicus_wheel wheel_prefix="front_left">
-            <origin xyz="${wheel_joint_x_abs} ${wheel_joint_y_abs} ${-wheel_joint_z_abs}" rpy="0 0 0" />
+            <origin xyz="${wheel_front_joint_x_abs} ${wheel_joint_y_abs} ${-wheel_joint_z_abs}" rpy="0 0 0" />
         </xacro:copernicus_wheel>
         <xacro:copernicus_wheel wheel_prefix="back_left">
-            <origin xyz="${-wheel_joint_x_abs} ${wheel_joint_y_abs} ${-wheel_joint_z_abs}" rpy="0 0 0" />
+            <origin xyz="${-wheel_back_joint_x_abs} ${wheel_joint_y_abs} ${-wheel_joint_z_abs}" rpy="0 0 0" />
         </xacro:copernicus_wheel>
         <!-- <gazebo>

File: copernicus_description/urdf/copernicus.xacro (robot description, xacro)
@@ -23,5 +23,5 @@
 SOFTWARE, EVEN IF ADVISED OF THE POSSIBILITY OF SUCH DAMAGE.
 -->
-<robot name="copernicus" xmlns:xacro="http://ros.org/wiki/xacro">
+<robot name="copernicus_robot" xmlns:xacro="http://ros.org/wiki/xacro">
   <xacro:include filename="$(find copernicus_description)/urdf/copernicus.urdf.xacro" />
   <xacro:copernicus_robot />

File: copernicus_description/urdf/vehicle_properties.xacro (robot description, xacro)
@@ -34,29 +34,22 @@
         <color rgba="0.5 0.5 0.5 1"/>
     </material>
-    <xacro:property name="chassis_mass" value="5.674"/>
-    <xacro:property name="chassis_l" value="0.75"/>
-    <xacro:property name="chassis_w" value="0.42"/>
-    <xacro:property name="chassis_h" value="0.23042"/>
-    <xacro:property name="chassis_h_no_susp" value="0.14"/>
-    <xacro:property name="chassis_t" value="0.003"/>
-    <xacro:property name="chassis_ixx" value="0.16120241795"/>
-    <xacro:property name="chassis_ixy" value="0.00001185952"/>
-    <xacro:property name="chassis_ixz" value="0.00001811354"/>
-    <xacro:property name="chassis_iyy" value="0.32866531087"/>
-    <xacro:property name="chassis_iyz" value="-0.000092298"/>
-    <xacro:property name="chassis_izz" value="0.449900533"/>
-    <xacro:property name="body_mass" value="10.7832"/>
-    <xacro:property name="body_h" value="0.15"/>
-    <xacro:property name="body_ixx" value="0.28969954739"/>
-    <xacro:property name="body_ixy" value="0.00014451398"/>
-    <xacro:property name="body_ixz" value="-0.02490442357"/>
-    <xacro:property name="body_iyy" value="0.4846882478"/>
-    <xacro:property name="body_iyz" value="0.0000035777"/>
-    <xacro:property name="body_izz" value="0.72198943224"/>
+    <xacro:property name="base_underside_h" value="0.20213"/>
+    <xacro:property name="base_mass" value="20.28"/>
+    <xacro:property name="base_l" value="0.76"/>
+    <xacro:property name="base_w" value="0.518"/>
+    <xacro:property name="base_h" value="0.387"/>
+    <xacro:property name="base_t" value="0.003"/>
+    <xacro:property name="base_ixx" value="1.25"/>
+    <xacro:property name="base_ixy" value="-0.00065"/>
+    <xacro:property name="base_ixz" value="0.064"/>
+    <xacro:property name="base_iyy" value="1.48"/>
+    <xacro:property name="base_iyz" value="-0.0167"/>
+    <xacro:property name="base_izz" value="1.15"/>
     <xacro:property name="wheel_width" value="0.1143" />
     <xacro:property name="wheel_radius" value="0.16938" />
-    <xacro:property name="wheel_joint_x_abs" value="0.28908" />
-    <xacro:property name="wheel_joint_y_abs" value="0.28858" />
-    <xacro:property name="wheel_joint_z_abs" value="0.04295" />
+    <xacro:property name="wheel_front_joint_x_abs" value="0.23337" />
+    <xacro:property name="wheel_joint_y_abs" value="0.259" />
+    <xacro:property name="wheel_joint_z_abs" value="0.03275" />
+    <xacro:property name="wheel_back_joint_x_abs" value="0.24988"/>
     <xacro:property name="wheel_ixx" value="0.036351442"/>
     <xacro:property name="wheel_ixy" value="0.000001230"/>
@@ -65,4 +58,18 @@
     <xacro:property name="wheel_iyz" value="0.0"/>
     <xacro:property name="wheel_izz" value="0.02162601213"/>
+    <xacro:property name="lidar_mount_l" value="0.537"/>
+    <xacro:property name="lidar_mount_w" value="0.075"/>
+    <xacro:property name="lidar_mount_t" value="0.075"/>
+    <xacro:property name="lidar_mount_mass" value="0.273"/>
+    <xacro:property name="lidar_mount_ixx" value="0.00693"/>
+    <xacro:property name="lidar_mount_ixy" value="0.0"/>
+    <xacro:property name="lidar_mount_ixz" value="0.0"/>
+    <xacro:property name="lidar_mount_iyy" value="0.000973"/>
+    <xacro:property name="lidar_mount_iyz" value="0.0"/>
+    <xacro:property name="lidar_mount_izz" value="0.00765"/>
+    <xacro:property name="lidar_mount_joint_x" value="0.38"/>
+    <xacro:property name="lidar_mount_joint_y" value="0.0"/>
+    <xacro:property name="lidar_mount_joint_z" value="0.025"/>
+    <xacro:property name="lidar_joint_x" value="0.04374"/>
     <xacro:property name="dummy_inertia" value="1e-09"/>
 </robot>

Commit message: Added dock to URDF

File: copernicus_description/urdf/accessories/camera.urdf.xacro (robot description, xacro)
@@ -30,5 +30,5 @@
             <parent link="base_link"/>
             <child link="${frame}"/>
-            <origin xyz="0 0 ${base_h}"/>
+            <origin xyz="${dock_joint_x - dock_l + 0.024/2} ${dock_joint_y} ${ dock_joint_z+dock_h/2+0.029/2 }" rpy="0 0 ${-PI}"/>
         </joint>
         <link name="${frame}">
@@ -36,5 +36,5 @@
                 <origin xyz="0 0 0" rpy="0 0 0"/>
                 <geometry>
-                    <box size="0.07 0.09 0.07"/>
+                    <box size="0.024 0.094 0.029"/>
                 </geometry>
             </visual>
@@ -42,5 +42,5 @@
                 <origin xyz="0 0 0" rpy="0 0 0"/>
                 <geometry>
-                    <box size="0.07 0.09 0.07"/>
+                    <box size="0.024 0.094 0.029"/>
                 </geometry>
             </collision>
@@ -57,5 +57,5 @@
                     <horizontal_fov>1.3962634</horizontal_fov>
                     <image>
-                        <width>1080</width>
+                        <width>1280</width>
                         <height>720</height>
                         <format>R8G8B8</format>

File: copernicus_description/urdf/copernicus.urdf.xacro (robot description, xacro)
@@ -34,4 +34,5 @@
     <xacro:arg name="imu_enabled" default="true"/>
     <xacro:arg name="gps_enabled" default="true"/>
+    <xacro:arg name="dock_enabled" default="true"/>
     <!-- TODO: Camera Mesh, Mount and Origin -->
     <xacro:arg name="camera_enabled" default="false"/>
@@ -78,4 +79,5 @@
             <origin xyz="${-wheel_back_joint_x_abs} ${wheel_joint_y_abs} ${-wheel_joint_z_abs}" rpy="0 0 0" />
         </xacro:copernicus_wheel>
+        <!-- FIX: Gazebo differential drive plugin not working -->
         <!-- <gazebo>
             <plugin name="gazebo_ros_control" filename="libgazebo_ros_control.so">
@@ -114,4 +116,11 @@
             <xacro:camera_></xacro:camera_>
         </xacro:if>
+        <!-- Dock -->
+        <xacro:if value="$(arg dock_enabled)">
+            <xacro:include filename="$(find copernicus_description)/urdf/accessories/dock.urdf.xacro"/>
+            <xacro:include filename="$(find copernicus_description)/urdf/accessories/camera.urdf.xacro"/>
+            <xacro:dock></xacro:dock>
+            <xacro:camera_></xacro:camera_>
+        </xacro:if>
     </xacro:macro>
 </robot>

File: copernicus_description/urdf/vehicle_properties.xacro (robot description, xacro)
@@ -72,4 +72,10 @@
     <xacro:property name="lidar_mount_joint_z" value="0.025"/>
     <xacro:property name="lidar_joint_x" value="0.04374"/>
+    <xacro:property name="dock_joint_x" value="-0.38"/>
+    <xacro:property name="dock_joint_y" value="0.0"/>
+    <xacro:property name="dock_joint_z" value="0.025"/>
+    <xacro:property name="dock_l" value="0.125"/>
+    <xacro:property name="dock_w" value="0.459"/>
+    <xacro:property name="dock_h" value="0.144"/>
     <xacro:property name="dummy_inertia" value="1e-09"/>
 </robot>
