Commit message: Renamed v2 URDF files

File: copernicus_description/urdf/accessories/camera.urdf.xacro (robot description, xacro)
@@ -30,5 +30,5 @@
             <parent link="base_link"/>
             <child link="${frame}"/>
-            <origin xyz="${dock_joint_x - dock_l + 0.024/2} ${dock_joint_y} ${ dock_joint_z+dock_h/2+0.029/2 }" rpy="0 0 ${-PI}"/>
+            <origin xyz="0 0 ${base_h}"/>
         </joint>
         <link name="${frame}">
@@ -36,5 +36,5 @@
                 <origin xyz="0 0 0" rpy="0 0 0"/>
                 <geometry>
-                    <box size="0.024 0.094 0.029"/>
+                    <box size="0.07 0.09 0.07"/>
                 </geometry>
             </visual>
@@ -42,5 +42,5 @@
                 <origin xyz="0 0 0" rpy="0 0 0"/>
                 <geometry>
-                    <box size="0.024 0.094 0.029"/>
+                    <box size="0.07 0.09 0.07"/>
                 </geometry>
             </collision>
@@ -57,5 +57,5 @@
                     <horizontal_fov>1.3962634</horizontal_fov>
                     <image>
-                        <width>1280</width>
+                        <width>1080</width>
                         <height>720</height>
                         <format>R8G8B8</format>

File: copernicus_description/urdf/accessories/imu.urdf.xacro (robot description, xacro)
@@ -29,5 +29,5 @@
             <parent link="base_link" />
             <child link="${frame}" />
-            <origin xyz="0 0 ${base_h/2}" rpy="0 0 0" />
+            <origin xyz="0 0 ${base_underside_h}" rpy="0 0 0" />
         </joint>
         <link name="${frame}">

File: copernicus_description/urdf/accessories/lidar.urdf.xacro (robot description, xacro)
@@ -28,5 +28,5 @@
                  min_angle:=-2.35619 max_angle:=2.35619 min_range:=0.5 max_range:=20.0 robot_namespace:=/">
       <joint name="lidar_mount_joint" type="fixed">
-          <origin xyz="${lidar_mount_joint_x} ${lidar_mount_joint_y} ${lidar_mount_joint_z}" rpy="0 0 0" />
+          <origin xyz="${lidar_mount_joint_x} ${lidar_mount_joint_y} ${lidar_mount_joint_z} " rpy="0 0 0" />
           <parent link="base_link" />
           <child link="lidar_mount" />
@@ -48,10 +48,10 @@
           <inertial>
               <origin xyz="0 0 0" rpy="0 0 0"/>
-              <mass value="0.1"/>
+              <mass value="${lidar_mount_mass}"/>
               <inertia ixx="${lidar_mount_ixx}" ixy="${lidar_mount_ixy}" ixz="${lidar_mount_ixz}" iyy="${lidar_mount_iyy}" iyz="${lidar_mount_iyz}" izz="${lidar_mount_izz}" />
           </inertial>
       </link>
       <joint name="lidar_joint" type="fixed">
-          <origin xyz="${lidar_joint_x} 0 0" rpy="${PI} 0 0" />
+          <origin xyz="${lidar_joint_x} ${lidar_joint_y} ${lidar_joint_z}" rpy="${PI} 0 0" />
           <parent link="lidar_mount" />
           <child link="${frame}" />

File: copernicus_description/urdf/copernicus.urdf.xacro (robot description, xacro)
@@ -34,13 +34,12 @@
     <xacro:arg name="imu_enabled" default="true"/>
     <xacro:arg name="gps_enabled" default="true"/>
-    <xacro:arg name="dock_enabled" default="true"/>
     <!-- TODO: Camera Mesh, Mount and Origin -->
     <xacro:arg name="camera_enabled" default="false"/>
-    <xacro:macro name="copernicus_base">
+    <xacro:macro name="copernicus_robot">
         <!-- Footprint -->
         <link name="footprint"/>
         <!-- Joint from footprint to base link(chassis) -->
         <joint name="base_footprint_joint" type="fixed">
-            <origin xyz="0 0 ${-base_underside_h}" rpy="0 0 0" />
+            <origin xyz="0 0 0.11457" rpy="0 0 0" />
             <parent link="base_link" />
             <child link="footprint" />
@@ -51,5 +50,5 @@
                 <origin xyz="0 0 0" rpy="0 0 0" />
                 <geometry>
-                    <mesh filename="package://copernicus_description/meshes/copernicus_v2.STL"/>
+                    <mesh filename="package://copernicus_description/meshes/copernicus.STL"/>
                 </geometry>
                 <material name="gray"/>
@@ -58,26 +57,25 @@
                 <origin xyz="0 0 0" rpy="0 0 0" />
                 <geometry>
-                    <mesh filename="package://copernicus_description/meshes/copernicus_v2.STL"/>
+                    <mesh filename="package://copernicus_description/meshes/copernicus.STL"/>
                 </geometry>
             </collision>
             <inertial>
-                <mass value="${ chassis_mass }"/>
-                <inertia ixx="${chassis_ixx}" ixy="${chassis_ixy}" ixz="${chassis_ixz}" iyy="${chassis_iyy}" iyz="${chassis_iyz}" izz="${chassis_izz}"/>
+                <mass value="${base_mass }"/>
+                <inertia ixx="${base_ixx}" ixy="${base_ixy}" ixz="${base_ixz}" iyy="${base_iyy}" iyz="${base_iyz}" izz="${base_izz}"/>
             </inertial>
         </link>
         <!-- Wheel -->
         <xacro:copernicus_wheel wheel_prefix="front_right">
-            <origin xyz="${wheel_front_joint_x_abs} ${-wheel_joint_y_abs} ${-wheel_joint_z_abs}" rpy="0 0 0" />
+            <origin xyz="${wheel_joint_x_abs} ${-wheel_joint_y_abs} ${-wheel_joint_z_abs}" rpy="0 0 0" />
         </xacro:copernicus_wheel>
         <xacro:copernicus_wheel wheel_prefix="back_right">
-            <origin xyz="${-wheel_back_joint_x_abs} ${-wheel_joint_y_abs} ${-wheel_joint_z_abs}" rpy="0 0 0" />
+            <origin xyz="${-wheel_joint_x_abs} ${-wheel_joint_y_abs} ${-wheel_joint_z_abs}" rpy="0 0 0" />
         </xacro:copernicus_wheel>
         <xacro:copernicus_wheel wheel_prefix="front_left">
-            <origin xyz="${wheel_front_joint_x_abs} ${wheel_joint_y_abs} ${-wheel_joint_z_abs}" rpy="0 0 0" />
+            <origin xyz="${wheel_joint_x_abs} ${wheel_joint_y_abs} ${-wheel_joint_z_abs}" rpy="0 0 0" />
         </xacro:copernicus_wheel>
         <xacro:copernicus_wheel wheel_prefix="back_left">
-            <origin xyz="${-wheel_back_joint_x_abs} ${wheel_joint_y_abs} ${-wheel_joint_z_abs}" rpy="0 0 0" />
+            <origin xyz="${-wheel_joint_x_abs} ${wheel_joint_y_abs} ${-wheel_joint_z_abs}" rpy="0 0 0" />
         </xacro:copernicus_wheel>
-        <!-- FIX: Gazebo differential drive plugin not working -->
         <!-- <gazebo>
             <plugin name="gazebo_ros_control" filename="libgazebo_ros_control.so">
@@ -116,11 +114,4 @@
             <xacro:camera_></xacro:camera_>
         </xacro:if>
-        <!-- Dock -->
-        <xacro:if value="$(arg dock_enabled)">
-            <xacro:include filename="$(find copernicus_description)/urdf/accessories/dock.urdf.xacro"/>
-            <xacro:include filename="$(find copernicus_description)/urdf/accessories/camera.urdf.xacro"/>
-            <xacro:dock></xacro:dock>
-            <xacro:camera_></xacro:camera_>
-        </xacro:if>
     </xacro:macro>
 </robot>

File: copernicus_description/urdf/copernicus.xacro (robot description, xacro)
@@ -23,5 +23,5 @@
 SOFTWARE, EVEN IF ADVISED OF THE POSSIBILITY OF SUCH DAMAGE.
 -->
-<robot name="copernicus_robot" xmlns:xacro="http://ros.org/wiki/xacro">
+<robot name="copernicus" xmlns:xacro="http://ros.org/wiki/xacro">
   <xacro:include filename="$(find copernicus_description)/urdf/copernicus.urdf.xacro" />
   <xacro:copernicus_robot />

File: copernicus_description/urdf/vehicle_properties.xacro (robot description, xacro)
@@ -34,22 +34,21 @@
         <color rgba="0.5 0.5 0.5 1"/>
     </material>
-    <xacro:property name="base_underside_h" value="0.20213"/>
-    <xacro:property name="base_mass" value="20.28"/>
-    <xacro:property name="base_l" value="0.76"/>
-    <xacro:property name="base_w" value="0.518"/>
-    <xacro:property name="base_h" value="0.387"/>
+    <xacro:property name="base_mass" value="5.674"/>
+    <xacro:property name="base_l" value="0.788"/>
+    <xacro:property name="base_w" value="0.715"/>
+    <xacro:property name="base_h" value="0.3795"/>
     <xacro:property name="base_t" value="0.003"/>
-    <xacro:property name="base_ixx" value="1.25"/>
-    <xacro:property name="base_ixy" value="-0.00065"/>
-    <xacro:property name="base_ixz" value="0.064"/>
-    <xacro:property name="base_iyy" value="1.48"/>
-    <xacro:property name="base_iyz" value="-0.0167"/>
-    <xacro:property name="base_izz" value="1.15"/>
+    <xacro:property name="base_ixx" value="1.729"/>
+    <xacro:property name="base_ixy" value="0.0051"/>
+    <xacro:property name="base_ixz" value="0.0435"/>
+    <xacro:property name="base_iyy" value="2.014"/>
+    <xacro:property name="base_iyz" value="0.0695"/>
+    <xacro:property name="base_izz" value="2.21"/>
+    <xacro:property name="base_underside_h" value="0.1025"/>
     <xacro:property name="wheel_width" value="0.1143" />
     <xacro:property name="wheel_radius" value="0.16938" />
-    <xacro:property name="wheel_front_joint_x_abs" value="0.23337" />
-    <xacro:property name="wheel_joint_y_abs" value="0.259" />
-    <xacro:property name="wheel_joint_z_abs" value="0.03275" />
-    <xacro:property name="wheel_back_joint_x_abs" value="0.24988"/>
+    <xacro:property name="wheel_joint_x_abs" value="0.21" />
+    <xacro:property name="wheel_joint_y_abs" value="0.3575" />
+    <xacro:property name="wheel_joint_z_abs" value="-0.05481" />
     <xacro:property name="wheel_ixx" value="0.036351442"/>
     <xacro:property name="wheel_ixy" value="0.000001230"/>
@@ -68,14 +67,10 @@
     <xacro:property name="lidar_mount_iyz" value="0.0"/>
     <xacro:property name="lidar_mount_izz" value="0.00765"/>
-    <xacro:property name="lidar_mount_joint_x" value="0.38"/>
+    <xacro:property name="lidar_mount_joint_x" value="0.394"/>
     <xacro:property name="lidar_mount_joint_y" value="0.0"/>
-    <xacro:property name="lidar_mount_joint_z" value="0.025"/>
-    <xacro:property name="lidar_joint_x" value="0.04374"/>
-    <xacro:property name="dock_joint_x" value="-0.38"/>
-    <xacro:property name="dock_joint_y" value="0.0"/>
-    <xacro:property name="dock_joint_z" value="0.025"/>
-    <xacro:property name="dock_l" value="0.125"/>
-    <xacro:property name="dock_w" value="0.459"/>
-    <xacro:property name="dock_h" value="0.144"/>
+    <xacro:property name="lidar_mount_joint_z" value="0.2195"/>
+    <xacro:property name="lidar_joint_x" value="0.075"/>
+    <xacro:property name="lidar_joint_y" value="0.0"/>
+    <xacro:property name="lidar_joint_z" value="0.05"/>
     <xacro:property name="dummy_inertia" value="1e-09"/>
 </robot>
