Commit message: Added Tim551 Mesh

File: copernicus_description/urdf/accessories/sick_tim_551.urdf.xacro (robot description, xacro)
@@ -25,6 +25,6 @@
 -->
 <robot name="copernicus" xmlns:xacro="https://ros.org/wiki/xacro">
-  <xacro:macro name="lidar" params="frame:=lidar topic:=scan_filtered sample_size:=720 update_rate:=50
-                 min_angle:=-1.57 max_angle:=1.57 min_range:=0.5 max_range:=20.0 robot_namespace:=/">
+  <xacro:macro name="lidar" params="frame:=lidar topic:=scan_filtered sample_size:=271 update_rate:=50
+                 min_angle:=-1.57 max_angle:=1.57 min_range:=0.05 max_range:=10.0 robot_namespace:=/">
       <joint name="lidar_mount_joint" type="fixed">
           <origin xyz="${lidar_mount_joint_x} ${lidar_mount_joint_y} ${lidar_mount_joint_z} " rpy="0 0 0" />
@@ -53,5 +53,5 @@
       </link>
       <joint name="lidar_joint" type="fixed">
-          <origin xyz="${lidar_joint_x} ${lidar_joint_y} ${lidar_joint_z}" rpy="0 0 0" />
+          <origin xyz="0.105 ${lidar_joint_y} -0.031" rpy="${PI} 0 0" />
           <parent link="lidar_mount" />
           <child link="${frame}" />
@@ -61,5 +61,5 @@
               <origin/>
               <geometry>
-                  <mesh filename="package://copernicus_description/meshes/hokuyo_ust10lx.STL"/>
+                  <mesh filename="package://copernicus_description/meshes/sick_tim551.stl"/>
               </geometry>
               <material name="gray"/>
@@ -68,5 +68,5 @@
               <origin xyz="0 0 0" rpy="0 0 0"/>
               <geometry>
-                <mesh filename="package://copernicus_description/meshes/hokuyo_ust10lx.STL"/>
+                <mesh filename="package://copernicus_description/meshes/sick_tim551.stl"/>
               </geometry>
           </collision>
@@ -74,11 +74,12 @@
               <origin xyz="0 0 0" rpy="0 0 0"/>
               <mass value="0.3"/>
-              <inertia ixx="${0.0833333 * 1.1 * (0.102*0.102 + 0.152*0.152)}" ixy="0.0" ixz="0.0"
-          iyy="${0.0833333 * 1.1 * (0.105*0.105 + 0.152*0.152)}" iyz="0.0"
-          izz="${0.0833333 * 1.1 * (0.105*0.105 + 0.102*0.102)}" />
+              <inertia ixx="${0.0833333 * 0.25 * (0.06*0.06 + 0.086*0.086)}" ixy="0.0" ixz="0.0"
+          iyy="${0.0833333 * 0.25 * (0.06*0.06 + 0.086*0.086)}" iyz="0.0"
+          izz="${0.0833333 * 0.25 * (0.06*0.06 + 0.06*0.06)}" />
           </inertial>
       </link>
       <gazebo reference="${frame}">
         <sensor type="ray" name="${frame}">
+          <always_on>true</always_on>
           <pose>0 0 0 0 0 0</pose>
           <visualize>false</visualize>
@@ -98,9 +99,4 @@
               <resolution>0.01</resolution>
             </range>
-            <noise>
-              <type>gaussian</type>
-              <mean>0.0</mean>
-              <stddev>0.001</stddev>
-            </noise>
           </ray>
           <plugin name="gazebo_ros_laser" filename="libgazebo_ros_laser.so">
@@ -108,4 +104,6 @@
             <frameName>${frame}</frameName>
             <robotNamespace>${robot_namespace}</robotNamespace>
+            <gaussianNoise>0.005</gaussianNoise>
+            <alwaysOn>true</alwaysOn>
           </plugin>
         </sensor>

File: copernicus_description/urdf/copernicus.urdf.xacro (robot description, xacro)
@@ -100,5 +100,5 @@
         <!-- LIDAR -->
         <xacro:if value="$(arg lidar_enabled)">
-            <xacro:include filename="$(find copernicus_description)/urdf/accessories/hokuyo_ust20lx.urdf.xacro"/>
+            <xacro:include filename="$(find copernicus_description)/urdf/accessories/sick_tim_551.urdf.xacro"/>
             <xacro:lidar></xacro:lidar>
         </xacro:if>
