Commit message: Updated Code to Work in Simulation

File: copernicus_description/urdf/accessories/gps.urdf.xacro (robot description, xacro)
@@ -25,5 +25,5 @@
 -->
 <robot name="copernicus" xmlns:xacro="https://ros.org/wiki/xacro">
-    <xacro:macro name="gps" params="frame:=gps topic:=gps/fix update_rate:=50 robot_namespace:=/ refLat:=1.345490 refLong:=103.682360">
+    <xacro:macro name="gps" params="frame:=gps topic:=gps/fix update_rate:=50 robot_namespace:=/ refLat:=1.3558320252002594 refLong:=103.6922425031662">
         <link name="${frame}">
             <inertial>

Commit message: Added Support for Multi Robot Navigation

File: copernicus_description/urdf/accessories/gps.urdf.xacro (robot description, xacro)
@@ -25,5 +25,5 @@
 -->
 <robot name="copernicus" xmlns:xacro="https://ros.org/wiki/xacro">
-    <xacro:macro name="gps" params="frame:=gps topic:=gps/fix update_rate:=50 robot_namespace:=/ refLat:=1.3558320252002594 refLong:=103.6922425031662">
+    <xacro:macro name="gps" params="frame:=gps topic:=gps/fix update_rate:=50 robot_namespace:=/ ref_latitude:=1.3558320252002594 ref_longitude:=103.6922425031662 tf_pre:=">
         <link name="${frame}">
             <inertial>
@@ -42,11 +42,11 @@
                 <updateRate>${update_rate}</updateRate>
                 <bodyName>${frame}</bodyName>
-                <frameId>${frame}</frameId>
+                <frameId>${tf_pre}${frame}</frameId>
                 <topicName>${topic}</topicName>
                 <velocityTopicName>${topic}_vel</velocityTopicName>
                 <driftFrequency>10.0 10.0 10.0</driftFrequency>
                 <drift>0.001 0.001 0.001</drift>
-                <referenceLatitude>${refLat}</referenceLatitude>
-                <referenceLongitude>${refLong}</referenceLongitude>
+                <referenceLatitude>${ref_latitude}</referenceLatitude>
+                <referenceLongitude>${ref_longitude}</referenceLongitude>
             </plugin>
         </gazebo>

File: copernicus_description/urdf/accessories/hokuyo_ust10lx.xacro (robot description, xacro)
@@ -81,4 +81,5 @@
       <gazebo reference="${frame}">
         <sensor type="ray" name="${frame}">
+          <always_on>true</always_on>
           <pose>0 0 0 0 0 0</pose>
           <visualize>false</visualize>
@@ -108,4 +109,6 @@
             <frameName>${frame}</frameName>
             <robotNamespace>${robot_namespace}</robotNamespace>
+            <gaussianNoise>0.005</gaussianNoise>
+            <alwaysOn>true</alwaysOn>
           </plugin>
         </sensor>

File: copernicus_description/urdf/accessories/imu.urdf.xacro (robot description, xacro)
@@ -25,5 +25,5 @@
 -->
 <robot name="copernicus" xmlns:xacro="https://ros.org/wiki/xacro">
-    <xacro:macro name="imu" params="frame:=imu topic:=imu/data update_rate:=50 robot_namespace:=/">
+    <xacro:macro name="imu" params="frame:=imu topic:=imu/data update_rate:=50 robot_namespace:=/ tf_pre:=">
         <joint name="${frame}_joint" type="fixed">
             <parent link="base_link" />
@@ -43,5 +43,5 @@
                 <updateRate>${update_rate}</updateRate>
                 <bodyName>${frame}</bodyName>
-                <frameId>${frame}</frameId>
+                <frameId>${tf_pre}${frame}</frameId>
                 <topicName>${topic}</topicName>
                 <accelDrift>0.005 0.005 0.005</accelDrift>

File: copernicus_description/urdf/components/wheel.urdf.xacro (robot description, xacro)
@@ -51,6 +51,8 @@
             <material>Gazebo/Black</material>
             <mu1 value="1.0"/>
-            <mu2 value="1.0"/><!--
-            <fdir1 value="1 0 0"/> -->
+            <mu2 value="1.0"/>
+            <kp value="10000000.0" />
+            <kd value="1.0" />
+            <fdir1 value="1 0 0"/>
         </gazebo>
         <!-- Wheel Joint -->
@@ -62,5 +64,5 @@
         </joint>
         <!-- Wheel Transmission -->
-        <transmission name="${wheel_prefix}_wheel_transmission">
+        <transmission name="${wheel_prefix}_wheel_transmission" type="SimpleTransmission">
             <type>transmission_interface/SimpleTransmission</type>
             <joint name="${wheel_prefix}_wheel_joint">
@@ -68,5 +70,4 @@
             </joint>
             <actuator name="${wheel_prefix}_motor">
-                <hardwareInterface>EffortJointInterface</hardwareInterface>
                 <mechanicalReduction>1</mechanicalReduction>
             </actuator>

File: copernicus_description/urdf/copernicus.urdf.xacro (robot description, xacro)
@@ -31,9 +31,13 @@
     <xacro:property name="PI" value="3.14159"/>
     <!-- xacro args -->
+    <xacro:arg name="robot_namespace" default="/" />
+    <xacro:arg name="tf_pre" default="" />
     <xacro:arg name="lidar_enabled" default="true"/>
     <xacro:arg name="imu_enabled" default="true"/>
     <xacro:arg name="gps_enabled" default="true"/>
+    <xacro:arg name="ref_latitude" default="0.0"/>
+    <xacro:arg name="ref_longitude" default="0.0"/>
     <xacro:arg name="camera_enabled" default="false"/>
-    <xacro:arg name="zed_camera_enabled" default="true"/>
+    <xacro:arg name="zed_camera_enabled" default="false"/>
     <xacro:macro name="copernicus_robot">
         <!-- Footprint -->
@@ -41,5 +45,5 @@
         <!-- Joint from footprint to base link(chassis) -->
         <joint name="base_footprint_joint" type="fixed">
-            <origin xyz="0 0 0.11457" rpy="0 0 0" />
+            <origin xyz="0 0 ${base_underside_h}" rpy="0 0 0" />
             <parent link="base_link" />
             <child link="footprint" />
@@ -78,17 +82,8 @@
             <origin xyz="${-wheel_joint_x_abs} ${wheel_joint_y_abs} ${-wheel_joint_z_abs}" rpy="0 0 0" />
         </xacro:copernicus_wheel>
-        <!-- <gazebo>
+        <gazebo>
             <plugin name="gazebo_ros_control" filename="libgazebo_ros_control.so">
-                <robotNamespace>/</robotNamespace>
-            </plugin>
-        </gazebo> -->
-        <gazebo>
-            <plugin name="omni_steering" filename="libgazebo_ros_planar_move.so">
-                <robotNamespace>/</robotNamespace>
-                <commandTopic>/cmd_vel</commandTopic>
-                <odometryTopic>odometry/wheel</odometryTopic>
-                <odometryFrame>odom</odometryFrame>
-                <odometryRate>30.0</odometryRate>
-                <robotBaseFrame>base_link</robotBaseFrame>
+                <robotNamespace>$(arg robot_namespace)</robotNamespace>
+                <robotSimType>gazebo_ros_control/DefaultRobotHWSim</robotSimType>
             </plugin>
         </gazebo>
@@ -96,5 +91,5 @@
         <xacro:if value="$(arg imu_enabled)">
             <xacro:include filename="$(find copernicus_description)/urdf/accessories/imu.urdf.xacro"/>
-            <xacro:imu></xacro:imu>
+            <xacro:imu robot_namespace="$(arg robot_namespace)" tf_pre="$(arg tf_pre)"></xacro:imu>
         </xacro:if>
         <!-- LIDAR -->
@@ -102,20 +97,20 @@
             <!-- <xacro:include filename="$(find copernicus_description)/urdf/accessories/hokuyo_ust20lx.urdf.xacro"/> -->
             <xacro:include filename="$(find copernicus_description)/urdf/accessories/lidar.urdf.xacro"/>
-            <xacro:lidar></xacro:lidar>
+            <xacro:lidar robot_namespace="$(arg robot_namespace)"></xacro:lidar>
         </xacro:if>
         <!-- GPS -->
         <xacro:if value="$(arg gps_enabled)">
             <xacro:include filename="$(find copernicus_description)/urdf/accessories/gps.urdf.xacro"/>
-            <xacro:gps></xacro:gps>
+            <xacro:gps robot_namespace="$(arg robot_namespace)" ref_latitude="$(arg ref_latitude)" ref_longitude="$(arg ref_longitude)" tf_pre="$(arg tf_pre)"></xacro:gps>
         </xacro:if>
         <!-- Camera -->
         <xacro:if value="$(arg camera_enabled)">
             <xacro:include filename="$(find copernicus_description)/urdf/accessories/camera.urdf.xacro"/>
-            <xacro:camera_></xacro:camera_>
+            <xacro:camera_ robot_namespace="$(arg robot_namespace)"></xacro:camera_>
         </xacro:if>
         <!-- ZED camera -->
         <xacro:if value="$(arg zed_camera_enabled)">
             <xacro:include filename="$(find copernicus_description)/urdf/accessories/camera.urdf.xacro"/>
-            <xacro:camera_ frame="zed_camera_center"></xacro:camera_>
+            <xacro:camera_ frame="zed_camera_center" robot_namespace="$(arg robot_namespace)"></xacro:camera_>
         </xacro:if>
     </xacro:macro>

File: copernicus_description/urdf/vehicle_properties.xacro (robot description, xacro)
@@ -45,5 +45,5 @@
     <xacro:property name="base_iyz" value="0.0695"/>
     <xacro:property name="base_izz" value="2.21"/>
-    <xacro:property name="base_underside_h" value="0.1025"/>
+    <xacro:property name="base_underside_h" value="0.11457"/>
     <xacro:property name="wheel_width" value="0.1143" />
     <xacro:property name="wheel_radius" value="0.16938" />
@@ -70,7 +70,7 @@
     <xacro:property name="lidar_mount_joint_y" value="0.0"/>
     <xacro:property name="lidar_mount_joint_z" value="0.2195"/>
-    <xacro:property name="lidar_joint_x" value="0.093"/>
+    <xacro:property name="lidar_joint_x" value="0.075"/>
     <xacro:property name="lidar_joint_y" value="0.0"/>
-    <xacro:property name="lidar_joint_z" value="-0.05"/>
+    <xacro:property name="lidar_joint_z" value="0.05"/>
     <xacro:property name="dummy_inertia" value="1e-09"/>
 </robot>
