Commit message: Added Velodyne Lidar and New Gazebo Map

File: copernicus_description/urdf/accessories/imu.urdf.xacro (robot description, xacro)
@@ -25,5 +25,5 @@
 -->
 <robot name="copernicus" xmlns:xacro="https://ros.org/wiki/xacro">
-    <xacro:macro name="imu" params="frame:=imu topic:=imu/data update_rate:=50 robot_namespace:=/ tf_pre:=">
+    <xacro:macro name="imu" params="frame:=imu topic:=imu/data update_rate:=10 robot_namespace:=/ tf_pre:=">
         <joint name="${frame}_joint" type="fixed">
             <parent link="base_link" />
@@ -38,18 +38,22 @@
             </inertial>
         </link>
-        <gazebo>
-            <plugin name="imu_plugin" filename="libhector_gazebo_ros_imu.so">
-                <robotNamespace>${robot_namespace}</robotNamespace>
-                <updateRate>${update_rate}</updateRate>
-                <bodyName>${frame}</bodyName>
-                <frameId>${tf_pre}${frame}</frameId>
-                <topicName>${topic}</topicName>
-                <accelDrift>0.005 0.005 0.005</accelDrift>
-                <accelGaussianNoise>0.005 0.005 0.005</accelGaussianNoise>
-                <rateDrift>0.005 0.005 0.005 </rateDrift>
-                <rateGaussianNoise>0.005 0.005 0.005</rateGaussianNoise>
-                <headingDrift>0.005</headingDrift>
-                <headingGaussianNoise>0.005</headingGaussianNoise>
-            </plugin>
+        <gazebo reference="${frame}">
+            <gravity>true</gravity>
+            <sensor name="imu_sensor" type="imu">
+                <always_on>true</always_on>
+                <update_rate>100</update_rate>
+                <visualize>true</visualize>
+                <topic>${topic}</topic>
+                <plugin filename="libgazebo_ros_imu_sensor.so" name="imu_plugin">
+                    <topicName>${topic}</topicName>
+                    <bodyName>${frame}</bodyName>
+                    <updateRateHZ>${update_rate}</updateRateHZ>
+                    <gaussianNoise>0.0</gaussianNoise>
+                    <xyzOffset>0 0 0</xyzOffset>
+                    <rpyOffset>0 0 0</rpyOffset>
+                    <frameName>base_link</frameName>
+                </plugin>
+                <pose>0 0 0 0 0 0</pose>
+            </sensor>
         </gazebo>
     </xacro:macro>

File: copernicus_description/urdf/copernicus.urdf.xacro (robot description, xacro)
@@ -33,5 +33,6 @@
     <xacro:arg name="robot_namespace" default="/" />
     <xacro:arg name="tf_pre" default="" />
-    <xacro:arg name="lidar_enabled" default="true"/>
+    <xacro:arg name="lidar_enabled" default="false"/>
+    <xacro:arg name="velodyne_enabled" default="true"/>
     <xacro:arg name="imu_enabled" default="true"/>
     <xacro:arg name="gps_enabled" default="true"/>
@@ -114,4 +115,10 @@
             <xacro:camera_ frame="zed_camera_center" robot_namespace="$(arg robot_namespace)"></xacro:camera_>
         </xacro:if>
+        <xacro:if value="$(arg velodyne_enabled)">
+            <xacro:include filename="$(find velodyne_description)/urdf/VLP-16.urdf.xacro"/>
+            <VLP-16 parent="base_link" name="velodyne" topic="velodyne_points" hz="10" samples="440" gpu="false">
+                <origin xyz="0.35 0 0.35" rpy="0 0.3 0" />
+            </VLP-16>
+        </xacro:if>
     </xacro:macro>
 </robot>
