Commit message: AUpdated URDF to V6.0

File: copernicus_description/urdf/accessories/lms_151.xacro (robot description, xacro)
@@ -25,16 +25,16 @@
 -->
 <robot name="copernicus" xmlns:xacro="https://ros.org/wiki/xacro">
-  <xacro:macro name="lidar" params="frame:=lidar topic:=scan_filtered sample_size:=720 update_rate:=50
-                 min_angle:=-1.57 max_angle:=1.57 min_range:=0.5 max_range:=10.0 robot_namespace:=/">
-      <joint name="lidar_mount_joint" type="fixed">
-          <origin xyz="${lidar_mount_joint_x} ${lidar_mount_joint_y} ${lidar_mount_joint_z} " rpy="0 0 0" />
+  <xacro:macro name="lms151" params="frame:=lms151 topic:=scan_filtered sample_size:=720 update_rate:=20
+                 min_angle:=-2.35619 max_angle:=2.35619 min_range:=0.5 max_range:=50.0 robot_namespace:=/">
+      <joint name="lms151_mount_joint" type="fixed">
+          <origin xyz="${lms151_mount_joint_x} ${lms151_mount_joint_y} ${lms151_mount_joint_z} " rpy="0 0 0" />
           <parent link="base_link" />
-          <child link="lidar_mount" />
+          <child link="lms151_mount" />
       </joint>
-      <link name="lidar_mount" type="fixed">
+      <link name="lms151_mount" type="fixed">
           <visual>
               <origin xyz="0 0 0" rpy="0 0 0"/>
               <geometry>
-                  <mesh filename="package://copernicus_description/meshes/lidar_mount.STL"/>
+                  <mesh filename="package://copernicus_description/meshes/lms_151_mount.STL"/>
                   <material name="gray"/>
               </geometry>
@@ -43,16 +43,16 @@
               <origin xyz="0 0 0" rpy="0 0 0"/>
               <geometry>
-                <mesh filename="package://copernicus_description/meshes/lidar_mount.STL"/>
+                <mesh filename="package://copernicus_description/meshes/lms_151_mount.STL"/>
               </geometry>
           </collision>
           <inertial>
               <origin xyz="0 0 0" rpy="0 0 0"/>
-              <mass value="${lidar_mount_mass}"/>
-              <inertia ixx="${lidar_mount_ixx}" ixy="${lidar_mount_ixy}" ixz="${lidar_mount_ixz}" iyy="${lidar_mount_iyy}" iyz="${lidar_mount_iyz}" izz="${lidar_mount_izz}" />
+              <mass value="${lms151_mount_mass}"/>
+              <inertia ixx="${lms151_mount_ixx}" ixy="${lms151_mount_ixy}" ixz="${lms151_mount_ixz}" iyy="${lms151_mount_iyy}" iyz="${lms151_mount_iyz}" izz="${lms151_mount_izz}" />
           </inertial>
       </link>
-      <joint name="lidar_joint" type="fixed">
-          <origin xyz="${lidar_joint_x} ${lidar_joint_y} ${lidar_joint_z}" rpy="0 0 0" />
-          <parent link="lidar_mount" />
+      <joint name="lms151_joint" type="fixed">
+          <origin xyz="${lms151_joint_x} ${lms151_joint_y} ${lms151_joint_z}" rpy="${PI} 0 0" />
+          <parent link="lms151_mount" />
           <child link="${frame}" />
       </joint>
@@ -61,5 +61,5 @@
               <origin/>
               <geometry>
-                  <mesh filename="package://copernicus_description/meshes/hokuyo_ust10lx.STL"/>
+                  <mesh filename="package://copernicus_description/meshes/lms_151.STL"/>
               </geometry>
               <material name="gray"/>
@@ -68,10 +68,10 @@
               <origin xyz="0 0 0" rpy="0 0 0"/>
               <geometry>
-                <mesh filename="package://copernicus_description/meshes/hokuyo_ust10lx.STL"/>
+                <mesh filename="package://copernicus_description/meshes/lms_151.STL"/>
               </geometry>
           </collision>
           <inertial>
               <origin xyz="0 0 0" rpy="0 0 0"/>
-              <mass value="0.3"/>
+              <mass value="1.1"/>
               <inertia ixx="${0.0833333 * 1.1 * (0.102*0.102 + 0.152*0.152)}" ixy="0.0" ixz="0.0"
           iyy="${0.0833333 * 1.1 * (0.105*0.105 + 0.152*0.152)}" iyz="0.0"
@@ -81,5 +81,4 @@
       <gazebo reference="${frame}">
         <sensor type="ray" name="${frame}">
-          <always_on>true</always_on>
           <pose>0 0 0 0 0 0</pose>
           <visualize>false</visualize>
@@ -109,6 +108,4 @@
             <frameName>${frame}</frameName>
             <robotNamespace>${robot_namespace}</robotNamespace>
-            <gaussianNoise>0.005</gaussianNoise>
-            <alwaysOn>true</alwaysOn>
           </plugin>
         </sensor>

File: copernicus_description/urdf/accessories/velodyne_mount.urdf.xacro (robot description, xacro)
@@ -25,36 +25,30 @@
 -->
 <robot name="copernicus" xmlns:xacro="https://ros.org/wiki/xacro">
-    <xacro:macro name="imu" params="frame:=imu topic:=imu/data update_rate:=10 robot_namespace:=/ tf_pre:=">
-        <joint name="${frame}_joint" type="fixed">
-            <parent link="base_link" />
-            <child link="${frame}" />
-            <origin xyz="0 0 ${ground_clearance}" rpy="0 0 0" />
-        </joint>
-        <link name="${frame}">
-            <inertial>
-                <mass value="0.001"/>
-                <origin xyz="0 0 0" rpy="0 0 0"/>
-                <inertia ixx="1e-09" ixy="0.0" ixz="0.0" iyy="1e-09" iyz="0.0" izz="1e-09"/>
-            </inertial>
-        </link>
-        <gazebo reference="${frame}">
-            <gravity>true</gravity>
-            <sensor name="imu_sensor" type="imu">
-                <always_on>true</always_on>
-                <update_rate>100</update_rate>
-                <visualize>true</visualize>
-                <topic>${topic}</topic>
-                <plugin filename="libgazebo_ros_imu_sensor.so" name="imu_plugin">
-                    <topicName>${topic}</topicName>
-                    <bodyName>${frame}</bodyName>
-                    <updateRateHZ>${update_rate}</updateRateHZ>
-                    <gaussianNoise>0.0</gaussianNoise>
-                    <xyzOffset>0 0 0</xyzOffset>
-                    <rpyOffset>0 0 0</rpyOffset>
-                    <frameName>base_link</frameName>
-                </plugin>
-                <pose>0 0 0 0 0 0</pose>
-            </sensor>
-        </gazebo>
-    </xacro:macro>
+  <xacro:macro name="velodyne_mount">
+      <joint name="velodyne_mount_joint" type="fixed">
+          <origin xyz="${velodyne_mount_joint_x} ${velodyne_mount_joint_y} ${velodyne_mount_joint_z} " rpy="0 ${velodyne_mount_joint_pitch} 0" />
+          <parent link="base_link" />
+          <child link="velodyne_mount" />
+      </joint>
+      <link name="velodyne_mount" type="fixed">
+          <visual>
+              <origin xyz="0 0 0" rpy="0 0 0"/>
+              <geometry>
+                  <mesh filename="package://copernicus_description/meshes/velodyne_mount.STL"/>
+                  <material name="gray"/>
+              </geometry>
+          </visual>
+          <collision>
+              <origin xyz="0 0 0" rpy="0 0 0"/>
+              <geometry>
+                <mesh filename="package://copernicus_description/meshes/velodyne_mount.STL"/>
+              </geometry>
+          </collision>
+          <inertial>
+              <origin xyz="0 0 0" rpy="0 0 0"/>
+              <mass value="${velodyne_mount_mass}"/>
+              <inertia ixx="${velodyne_mount_ixx}" ixy="${velodyne_mount_ixy}" ixz="${velodyne_mount_ixz}" iyy="${velodyne_mount_iyy}" iyz="${velodyne_mount_iyz}" izz="${velodyne_mount_izz}" />
+          </inertial>
+      </link>
+  </xacro:macro>
 </robot>

File: copernicus_description/urdf/components/wheel.urdf.xacro (robot description, xacro)
@@ -30,5 +30,5 @@
         <link name="${wheel_prefix}_wheel">
             <visual>
-                <origin xyz="0 0 0" rpy="0 0 ${PI/2}"/>
+                <origin xyz="0 0 0" rpy="0 0 0"/>
                 <geometry>
                     <mesh filename="package://copernicus_description/meshes/wheel.STL"/>

File: copernicus_description/urdf/copernicus.urdf.xacro (robot description, xacro)
@@ -1,5 +1,5 @@
 <?xml version="1.0"?>
 <!--
-Copyright (c) 2017, Botsync Pte. Ltd.
+Copyright (c) 2019, Botsync Pte. Ltd.
 All rights reserved.
 Redistribution and use in source and binary forms, with or without
@@ -41,5 +41,5 @@
     <xacro:arg name="camera_enabled" default="false"/>
     <xacro:arg name="zed_camera_enabled" default="false"/>
-    <xacro:arg name="guide_sensor_enabled" default="true"/>
+    <xacro:arg name="guide_sensor_enabled" default="false"/>
     <xacro:macro name="copernicus_robot">
         <!-- Footprint -->
@@ -47,5 +47,5 @@
         <!-- Joint from footprint to base link(chassis) -->
         <joint name="base_footprint_joint" type="fixed">
-            <origin xyz="0 0 ${base_underside_h}" rpy="0 0 0" />
+            <origin xyz="0 0 ${ground_clearance}" rpy="0 0 0" />
             <parent link="base_link" />
             <child link="footprint" />
@@ -56,5 +56,5 @@
                 <origin xyz="0 0 0" rpy="0 0 0" />
                 <geometry>
-                    <mesh filename="package://copernicus_description/meshes/copernicus_v4.STL"/>
+                    <mesh filename="package://copernicus_description/meshes/copernicus.STL"/>
                 </geometry>
                 <material name="gray"/>
@@ -63,5 +63,5 @@
                 <origin xyz="0 0 0" rpy="0 0 0" />
                 <geometry>
-                    <mesh filename="package://copernicus_description/meshes/copernicus_v4.STL"/>
+                    <mesh filename="package://copernicus_description/meshes/copernicus.STL"/>
                 </geometry>
             </collision>
@@ -72,8 +72,8 @@
         </link>
         <!-- Wheel -->
-        <xacro:copernicus_wheel wheel_prefix="front_right"><origin xyz="${wheel_joint_x_abs} ${-wheel_joint_y_abs} ${-wheel_joint_z_abs}" rpy="0 0 0"/></xacro:copernicus_wheel>
-        <xacro:copernicus_wheel wheel_prefix="back_right"><origin xyz="${-wheel_joint_x_abs} ${-wheel_joint_y_abs} ${-wheel_joint_z_abs}" rpy="0 0 0"/></xacro:copernicus_wheel>
-        <xacro:copernicus_wheel wheel_prefix="front_left"><origin xyz="${wheel_joint_x_abs} ${wheel_joint_y_abs} ${-wheel_joint_z_abs}" rpy="0 0 0"/></xacro:copernicus_wheel>
-        <xacro:copernicus_wheel wheel_prefix="back_left"><origin xyz="${-wheel_joint_x_abs} ${wheel_joint_y_abs} ${-wheel_joint_z_abs}" rpy="0 0 0"/></xacro:copernicus_wheel>
+        <xacro:copernicus_wheel wheel_prefix="front_right"><origin xyz="${wheel_joint_x_abs} ${-wheel_joint_y_abs} ${wheel_joint_z_abs}" rpy="0 0 0"/></xacro:copernicus_wheel>
+        <xacro:copernicus_wheel wheel_prefix="back_right"><origin xyz="${-wheel_joint_x_abs} ${-wheel_joint_y_abs} ${wheel_joint_z_abs}" rpy="0 0 0"/></xacro:copernicus_wheel>
+        <xacro:copernicus_wheel wheel_prefix="front_left"><origin xyz="${wheel_joint_x_abs} ${wheel_joint_y_abs} ${wheel_joint_z_abs}" rpy="0 0 0"/></xacro:copernicus_wheel>
+        <xacro:copernicus_wheel wheel_prefix="back_left"><origin xyz="${-wheel_joint_x_abs} ${wheel_joint_y_abs} ${wheel_joint_z_abs}" rpy="0 0 0"/></xacro:copernicus_wheel>
         <gazebo>
             <plugin name="gazebo_ros_control" filename="libgazebo_ros_control.so">
@@ -87,9 +87,8 @@
             <xacro:imu robot_namespace="$(arg robot_namespace)" tf_pre="$(arg tf_pre)"></xacro:imu>
         </xacro:if>
-        <!-- LIDAR -->
+        <!-- LMS151 -->
         <xacro:if value="$(arg lidar_enabled)">
-            <!-- <xacro:include filename="$(find copernicus_description)/urdf/accessories/hokuyo_ust20lx.urdf.xacro"/> -->
-            <xacro:include filename="$(find copernicus_description)/urdf/accessories/lidar.urdf.xacro"/>
-            <xacro:lidar robot_namespace="$(arg robot_namespace)"></xacro:lidar>
+            <xacro:include filename="$(find copernicus_description)/urdf/accessories/lms151.urdf.xacro"/>
+            <xacro:lms151 robot_namespace="$(arg robot_namespace)"></xacro:lms151>
         </xacro:if>
         <!-- GPS -->
@@ -108,8 +107,11 @@
             <xacro:camera_ frame="zed_camera_center" robot_namespace="$(arg robot_namespace)"></xacro:camera_>
         </xacro:if>
+        <!-- Velodyne -->
         <xacro:if value="$(arg velodyne_enabled)">
+            <xacro:include filename="$(find copernicus_description)/urdf/accessories/velodyne_mount.urdf.xacro"/>
+            <xacro:velodyne_mount></xacro:velodyne_mount>
             <xacro:include filename="$(find velodyne_description)/urdf/VLP-16.urdf.xacro"/>
-            <VLP-16 parent="base_link" name="velodyne" topic="velodyne_points" hz="10" samples="440" gpu="false" min_range="0.2">
-                <origin xyz="0.38685 0 0.41478" rpy="0.0 0.20944 0" />
+            <VLP-16 parent="velodyne_mount" name="velodyne" topic="velodyne_points" hz="10" samples="440" gpu="false" min_range="0.2">
+                <origin xyz="${velodyne_joint_x} ${velodyne_joint_y} ${velodyne_joint_z}" rpy="0 ${-velodyne_joint_pitch} 0" />
             </VLP-16>
         </xacro:if>

File: copernicus_description/urdf/vehicle_properties.xacro (robot description, xacro)
@@ -35,42 +35,59 @@
     </material>
     <xacro:property name="base_mass" value="5.674"/>
-    <xacro:property name="base_l" value="0.788"/>
-    <xacro:property name="base_w" value="0.715"/>
-    <xacro:property name="base_h" value="0.3795"/>
-    <xacro:property name="base_t" value="0.003"/>
-    <xacro:property name="base_ixx" value="1.729"/>
-    <xacro:property name="base_ixy" value="0.0051"/>
-    <xacro:property name="base_ixz" value="0.0435"/>
-    <xacro:property name="base_iyy" value="2.014"/>
-    <xacro:property name="base_iyz" value="0.0695"/>
-    <xacro:property name="base_izz" value="2.21"/>
-    <xacro:property name="base_underside_h" value="0.11457"/>
-    <xacro:property name="wheel_width" value="0.1143" />
-    <xacro:property name="wheel_radius" value="0.16938" />
-    <xacro:property name="wheel_joint_x_abs" value="0.21" />
-    <xacro:property name="wheel_joint_y_abs" value="0.3575" />
-    <xacro:property name="wheel_joint_z_abs" value="-0.05481" />
-    <xacro:property name="wheel_ixx" value="0.036351442"/>
-    <xacro:property name="wheel_ixy" value="0.000001230"/>
-    <xacro:property name="wheel_ixz" value="0.0"/>
-    <xacro:property name="wheel_iyy" value="0.021626014"/>
-    <xacro:property name="wheel_iyz" value="0.0"/>
-    <xacro:property name="wheel_izz" value="0.02162601213"/>
-    <xacro:property name="lidar_mount_l" value="0.537"/>
-    <xacro:property name="lidar_mount_w" value="0.075"/>
-    <xacro:property name="lidar_mount_t" value="0.075"/>
-    <xacro:property name="lidar_mount_mass" value="0.273"/>
-    <xacro:property name="lidar_mount_ixx" value="0.00693"/>
-    <xacro:property name="lidar_mount_ixy" value="0.0"/>
-    <xacro:property name="lidar_mount_ixz" value="0.0"/>
-    <xacro:property name="lidar_mount_iyy" value="0.000973"/>
-    <xacro:property name="lidar_mount_iyz" value="0.0"/>
-    <xacro:property name="lidar_mount_izz" value="0.00765"/>
-    <xacro:property name="lidar_mount_joint_x" value="0.394"/>
-    <xacro:property name="lidar_mount_joint_y" value="0.0"/>
-    <xacro:property name="lidar_mount_joint_z" value="0.2195"/>
-    <xacro:property name="lidar_joint_x" value="0.075"/>
-    <xacro:property name="lidar_joint_y" value="0.0"/>
-    <xacro:property name="lidar_joint_z" value="0.05"/>
+    <xacro:property name="base_l" value="0.646"/>
+    <xacro:property name="base_w" value="0.456"/>
+    <xacro:property name="base_h" value="0.323"/>
+    <xacro:property name="base_ixx" value="3.28"/>
+    <xacro:property name="base_ixy" value="0.00"/>
+    <xacro:property name="base_ixz" value="0.00"/>
+    <xacro:property name="base_iyy" value="3.69"/>
+    <xacro:property name="base_iyz" value="0.00"/>
+    <xacro:property name="base_izz" value="2.26"/>
+    <xacro:property name="ground_clearance" value="0.11457"/>
+    <xacro:property name="wheel_width" value="0.120" />
+    <xacro:property name="wheel_radius" value="0.18" />
+    <xacro:property name="wheel_joint_x_abs" value="0.22030" />
+    <xacro:property name="wheel_joint_y_abs" value="0.29490" />
+    <xacro:property name="wheel_joint_z_abs" value="0.07300" />
+    <xacro:property name="wheel_ixx" value="0.739"/>
+    <xacro:property name="wheel_ixy" value="0.170"/>
+    <xacro:property name="wheel_ixz" value="0.236"/>
+    <xacro:property name="wheel_iyy" value="0.741"/>
+    <xacro:property name="wheel_iyz" value="0.299"/>
+    <xacro:property name="wheel_izz" value="0.460"/>
+    <xacro:property name="lms151_mount_l" value="0.156"/>
+    <xacro:property name="lms151_mount_h" value="0.094"/>
+    <xacro:property name="lms151_mount_w" value="0.1102"/>
+    <xacro:property name="lms151_mount_mass" value="0.229"/>
+    <xacro:property name="lms151_mount_ixx" value="0.002"/>
+    <xacro:property name="lms151_mount_ixy" value="0.000"/>
+    <xacro:property name="lms151_mount_ixz" value="0.000"/>
+    <xacro:property name="lms151_mount_iyy" value="0.005"/>
+    <xacro:property name="lms151_mount_iyz" value="0.000"/>
+    <xacro:property name="lms151_mount_izz" value="0.002"/>
+    <xacro:property name="lms151_mount_joint_x" value="0.099"/>
+    <xacro:property name="lms151_mount_joint_y" value="0"/>
+    <xacro:property name="lms151_mount_joint_z" value="0.042"/>
+    <xacro:property name="lms151_joint_x" value="0.027"/>
+    <xacro:property name="lms151_joint_y" value="0.0625"/>
+    <xacro:property name="lms151_joint_z" value="0.03"/>
+    <xacro:property name="velodyne_mount_l" value="0.112"/>
+    <xacro:property name="velodyne_mount_h" value="0.039"/>
+    <xacro:property name="velodyne_mount_w" value="0.125"/>
+    <xacro:property name="velodyne_mount_mass" value="0.300"/>
+    <xacro:property name="velodyne_mount_ixx" value="0.002"/>
+    <xacro:property name="velodyne_mount_ixy" value="0.000"/>
+    <xacro:property name="velodyne_mount_ixz" value="0.000"/>
+    <xacro:property name="velodyne_mount_iyy" value="0.005"/>
+    <xacro:property name="velodyne_mount_iyz" value="0.000"/>
+    <xacro:property name="velodyne_mount_izz" value="0.002"/>
+    <xacro:property name="velodyne_mount_joint_x" value="0.259"/>
+    <xacro:property name="velodyne_mount_joint_y" value="-0.0625"/>
+    <xacro:property name="velodyne_mount_joint_z" value="0.296"/>
+    <xacro:property name="velodyne_mount_joint_pitch" value="0.415"/>
+    <xacro:property name="velodyne_joint_x" value="0.027"/>
+    <xacro:property name="velodyne_joint_y" value="0.0625"/>
+    <xacro:property name="velodyne_joint_z" value="0.03"/>
+    <xacro:property name="velodyne_joint_pitch" value="0.262"/>
     <xacro:property name="dummy_inertia" value="1e-09"/>
 </robot>
