Commit message: Copernicus release update.

File: copernicus_description/urdf/accessories/lms_151_copernicus.urdf.xacro (robot description, xacro)
@@ -36,5 +36,5 @@
               <origin xyz="0 0 0" rpy="0 0 0"/>
               <geometry>
-                  <mesh filename="package://copernicus_description/meshes/lms_151_mount.dae"/>
+                  <mesh filename="package://copernicus_description/meshes/lms_151_mount.dae" scale="0.1 0.1 0.1"/>
                   <material name="gray"/>
               </geometry>
@@ -43,5 +43,5 @@
               <origin xyz="0 0 0" rpy="0 0 0"/>
               <geometry>
-                <mesh filename="package://copernicus_description/meshes/lms_151_mount.dae"/>
+                <mesh filename="package://copernicus_description/meshes/lms_151_mount.dae" scale="0.1 0.1 0.1"/>
               </geometry>
           </collision>
@@ -53,5 +53,5 @@
       </link>
       <joint name="lms151_joint" type="fixed">
-          <origin xyz="${lms151_joint_x} ${lms151_joint_y} ${lms151_joint_z}" rpy="${PI} 0 0" />
+          <origin xyz="${lms151_joint_x} ${lms151_joint_y} ${lms151_joint_z}" rpy="0 0 0" />
           <parent link="lms151_mount" />
           <child link="${frame}" />
@@ -61,5 +61,5 @@
               <origin xyz="0 0 0" rpy="0 0 0"/>-->
               <geometry>
-                  <mesh filename="package://copernicus_description/meshes/lms_151.dae"/>
+                  <mesh filename="package://copernicus_description/meshes/lms_151.dae" scale="0.1 0.1 0.1"/>
               </geometry>
               <material name="gray"/>
@@ -68,5 +68,5 @@
               <origin xyz="0 0 0" rpy="0 0 0"/>
               <geometry>
-                <mesh filename="package://copernicus_description/meshes/lms_151.dae"/>
+                <mesh filename="package://copernicus_description/meshes/lms_151.dae" scale="0.1 0.1 0.1"/>
               </geometry>
           </collision>

File: copernicus_description/urdf/copernicus.urdf.xacro (robot description, xacro)
@@ -32,8 +32,9 @@
     <!-- xacro args -->
     <xacro:arg name="robot_namespace" default="/" />
-    <xacro:arg name="lidar_enabled" default="true"/>
+    <xacro:arg name="lidar_enabled" default="false"/>
+    <xacro:arg name="test_lidar_enabled" default="true"/>
     <xacro:arg name="sick_lms151_enabled" default="false"/>
     <xacro:arg name="velodyne_enabled" default="false"/>
-    <xacro:arg name="imu_enabled" default="false"/>
+    <xacro:arg name="imu_enabled" default="true"/>
     <!--<xacro:arg name="camera_enabled" default="false"/>
     <xacro:arg name="intel_d435i_enabled" default="false"/>-->
@@ -90,4 +91,9 @@
             <xacro:lidar sick_lms151_enabled="$(arg sick_lms151_enabled)" robot_namespace="$(arg robot_namespace)"></xacro:lidar>
         </xacro:if>
+        <!-- TEST LIDAR -->
+        <xacro:if value="$(arg test_lidar_enabled)">
+            <xacro:include filename="$(find copernicus_description)/urdf/accessories/lidar_copernicus.urdf.xacro"/>
+            <xacro:lidar robot_namespace="$(arg robot_namespace)"></xacro:lidar>
+        </xacro:if>
         <!-- Velodyne -->
         <xacro:if value="$(arg velodyne_enabled)">

File: copernicus_description/urdf/vehicle_properties.xacro (robot description, xacro)
@@ -66,10 +66,13 @@
     <xacro:property name="lms151_mount_iyz" value="0.000"/>
     <xacro:property name="lms151_mount_izz" value="0.002"/>
-    <xacro:property name="lms151_mount_joint_x" value="0.0177"/>
+    <xacro:property name="lms151_mount_joint_x" value="0.0"/>
     <xacro:property name="lms151_mount_joint_y" value="0.0"/>
-    <xacro:property name="lms151_mount_joint_z" value="0.356"/>
-    <xacro:property name="lms151_joint_x" value="0.0453"/>
+    <xacro:property name="lms151_mount_joint_z" value="0.4155"/>
+    <xacro:property name="lms151_joint_x" value="0.0"/>
     <xacro:property name="lms151_joint_y" value="0.0"/>
-    <xacro:property name="lms151_joint_z" value="0.158"/>
+    <xacro:property name="lms151_joint_z" value="0.0"/>
+    <!-- base of lidar mopunt, x position in lidar_copernicus.urdf.xacro -->
+    <xacro:property name="lidar_joint_y" value="0.0"/>
+    <xacro:property name="lidar_joint_z" value="0.395"/>
     <xacro:property name="velodyne_mount_l" value="0.112"/>
     <xacro:property name="velodyne_mount_h" value="0.039"/>
