Commit message: Changed LIDAR

File: copernicus_description/urdf/copernicus.urdf.xacro (robot description, xacro)
@@ -100,5 +100,5 @@
         <!-- LIDAR -->
         <xacro:if value="$(arg lidar_enabled)">
-            <xacro:include filename="$(find copernicus_description)/urdf/accessories/lidar.urdf.xacro"/>
+            <xacro:include filename="$(find copernicus_description)/urdf/accessories/hokuyo_ust20lx.urdf.xacro"/>
             <xacro:lidar></xacro:lidar>
         </xacro:if>

File: copernicus_description/urdf/vehicle_properties.xacro (robot description, xacro)
@@ -70,7 +70,7 @@
     <xacro:property name="lidar_mount_joint_y" value="0.0"/>
     <xacro:property name="lidar_mount_joint_z" value="0.2195"/>
-    <xacro:property name="lidar_joint_x" value="0.075"/>
+    <xacro:property name="lidar_joint_x" value="0.093"/>
     <xacro:property name="lidar_joint_y" value="0.0"/>
-    <xacro:property name="lidar_joint_z" value="0.05"/>
+    <xacro:property name="lidar_joint_z" value="-0.05"/>
     <xacro:property name="dummy_inertia" value="1e-09"/>
 </robot>

Commit message: Updated URDF Files

File: copernicus_description/urdf/copernicus.urdf.xacro (robot description, xacro)
@@ -55,5 +55,5 @@
                 <origin xyz="0 0 0" rpy="0 0 0" />
                 <geometry>
-                    <mesh filename="package://copernicus_description/meshes/copernicus.STL"/>
+                    <mesh filename="package://copernicus_description/meshes/copernicus_v4.STL"/>
                 </geometry>
                 <material name="gray"/>
@@ -62,25 +62,17 @@
                 <origin xyz="0 0 0" rpy="0 0 0" />
                 <geometry>
-                    <mesh filename="package://copernicus_description/meshes/copernicus.STL"/>
+                    <mesh filename="package://copernicus_description/meshes/copernicus_v4.STL"/>
                 </geometry>
             </collision>
             <inertial>
-                <mass value="${base_mass }"/>
+                <mass value="${base_mass}"/>
                 <inertia ixx="${base_ixx}" ixy="${base_ixy}" ixz="${base_ixz}" iyy="${base_iyy}" iyz="${base_iyz}" izz="${base_izz}"/>
             </inertial>
         </link>
         <!-- Wheel -->
-        <xacro:copernicus_wheel wheel_prefix="front_right">
-            <origin xyz="${wheel_joint_x_abs} ${-wheel_joint_y_abs} ${-wheel_joint_z_abs}" rpy="0 0 0" />
-        </xacro:copernicus_wheel>
-        <xacro:copernicus_wheel wheel_prefix="back_right">
-            <origin xyz="${-wheel_joint_x_abs} ${-wheel_joint_y_abs} ${-wheel_joint_z_abs}" rpy="0 0 0" />
-        </xacro:copernicus_wheel>
-        <xacro:copernicus_wheel wheel_prefix="front_left">
-            <origin xyz="${wheel_joint_x_abs} ${wheel_joint_y_abs} ${-wheel_joint_z_abs}" rpy="0 0 0" />
-        </xacro:copernicus_wheel>
-        <xacro:copernicus_wheel wheel_prefix="back_left">
-            <origin xyz="${-wheel_joint_x_abs} ${wheel_joint_y_abs} ${-wheel_joint_z_abs}" rpy="0 0 0" />
-        </xacro:copernicus_wheel>
+        <xacro:copernicus_wheel wheel_prefix="front_right"><origin xyz="${wheel_joint_x_abs} ${-wheel_joint_y_abs} ${-wheel_joint_z_abs}" rpy="0 0 0"/></xacro:copernicus_wheel>
+        <xacro:copernicus_wheel wheel_prefix="back_right"><origin xyz="${-wheel_joint_x_abs} ${-wheel_joint_y_abs} ${-wheel_joint_z_abs}" rpy="0 0 0"/></xacro:copernicus_wheel>
+        <xacro:copernicus_wheel wheel_prefix="front_left"><origin xyz="${wheel_joint_x_abs} ${wheel_joint_y_abs} ${-wheel_joint_z_abs}" rpy="0 0 0"/></xacro:copernicus_wheel>
+        <xacro:copernicus_wheel wheel_prefix="back_left"><origin xyz="${-wheel_joint_x_abs} ${wheel_joint_y_abs} ${-wheel_joint_z_abs}" rpy="0 0 0"/></xacro:copernicus_wheel>
         <gazebo>
             <plugin name="gazebo_ros_control" filename="libgazebo_ros_control.so">
@@ -118,5 +110,5 @@
             <xacro:include filename="$(find velodyne_description)/urdf/VLP-16.urdf.xacro"/>
             <VLP-16 parent="base_link" name="velodyne" topic="velodyne_points" hz="10" samples="440" gpu="false">
-                <origin xyz="0.35 0 0.35" rpy="0 0.3 0" />
+                <origin xyz="0.38685 0 0.41478" rpy="0.0 0.20944 0" />
             </VLP-16>
         </xacro:if>

Commit message: Updated LMS Mount URDF

File: copernicus_description/urdf/copernicus.urdf.xacro (robot description, xacro)
@@ -89,5 +89,5 @@
         <!-- LMS151 -->
         <xacro:if value="$(arg lidar_enabled)">
-            <xacro:include filename="$(find copernicus_description)/urdf/accessories/lms151.urdf.xacro"/>
+            <xacro:include filename="$(find copernicus_description)/urdf/accessories/lms_151.urdf.xacro"/>
             <xacro:lms151 robot_namespace="$(arg robot_namespace)"></xacro:lms151>
         </xacro:if>

File: copernicus_description/urdf/vehicle_properties.xacro (robot description, xacro)
@@ -66,10 +66,10 @@
     <xacro:property name="lms151_mount_iyz" value="0.000"/>
     <xacro:property name="lms151_mount_izz" value="0.002"/>
-    <xacro:property name="lms151_mount_joint_x" value="0.099"/>
+    <xacro:property name="lms151_mount_joint_x" value="0.0177"/>
     <xacro:property name="lms151_mount_joint_y" value="0"/>
-    <xacro:property name="lms151_mount_joint_z" value="0.042"/>
-    <xacro:property name="lms151_joint_x" value="0.027"/>
-    <xacro:property name="lms151_joint_y" value="0.0625"/>
-    <xacro:property name="lms151_joint_z" value="0.03"/>
+    <xacro:property name="lms151_mount_joint_z" value="0.356"/>
+    <xacro:property name="lms151_joint_x" value="0.0453"/>
+    <xacro:property name="lms151_joint_y" value="0.0"/>
+    <xacro:property name="lms151_joint_z" value="0.158"/>
     <xacro:property name="velodyne_mount_l" value="0.112"/>
     <xacro:property name="velodyne_mount_h" value="0.039"/>
@@ -88,5 +88,5 @@
     <xacro:property name="velodyne_joint_x" value="0.027"/>
     <xacro:property name="velodyne_joint_y" value="0.0625"/>
-    <xacro:property name="velodyne_joint_z" value="0.03"/>
+    <xacro:property name="velodyne_joint_z" value="0.0295"/>
     <xacro:property name="velodyne_joint_pitch" value="0.262"/>
     <xacro:property name="dummy_inertia" value="1e-09"/>
