Commit message: Fixed URDF Bug

File: copernicus_description/urdf/accessories_v2/lidar.urdf.xacro (robot description, xacro)
@@ -25,5 +25,5 @@
 -->
 <robot name="copernicus" xmlns:xacro="https://ros.org/wiki/xacro">
-  <xacro:macro name="lidar" params="frame:=lidar topic:=scan sample_size:=720 update_rate:=50
+  <xacro:macro name="lidar" params="frame:=lidar topic:=scan_filtered sample_size:=720 update_rate:=50
                  min_angle:=-2.35619 max_angle:=2.35619 min_range:=0.5 max_range:=20.0 robot_namespace:=/">
       <joint name="lidar_mount_joint" type="fixed">

File: copernicus_description/urdf/copernicus_v2.urdf.xacro (robot description, xacro)
@@ -42,6 +42,6 @@
         <joint name="base_footprint_joint" type="fixed">
             <origin xyz="0 0 0.11457" rpy="0 0 0" />
-            <parent link="footprint" />
-            <child link="base_link" />
+            <parent link="base_link" />
+            <child link="footprint" />
         </joint>
         <!-- Chassis a.k.a base_link -->
